File: CAN.kicad_sch (KiCad schematic)
At the start: 9 parts

Commit message: rename; annotate and import to pcb
Parts:
- gave numbers to parts that had none: 9
Changed lines of the file:
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@@
   (symbol (lib_id "Connector:TestPoint_Small") (at 129.286 126.238 0) (unit 1)
     (in_bom yes) (on_board yes)
-    (property "Reference" "TP?" (id 0) (at 128.016 124.714 0)
+    (property "Reference" "TP5" (id 0) (at 128.016 124.714 0)
       (effects (font (size 1.27 1.27)) (justify left))
     )
@@
   (symbol (lib_id "Device:Crystal_GND24_Small") (at 212.598 69.088 90) (unit 1)
     (in_bom yes) (on_board yes)
-    (property "Reference" "Y?" (id 0) (at 209.423 65.913 90)
+    (property "Reference" "Y1" (id 0) (at 209.423 65.913 90)
       (effects (font (size 1.27 1.27)) (justify right))
     )
@@
   (symbol (lib_id "Connector:TestPoint_Small") (at 175.768 95.504 0) (unit 1)
     (in_bom yes) (on_board yes)
-    (property "Reference" "TP?" (id 0) (at 174.117 97.282 0)
+    (property "Reference" "TP6" (id 0) (at 174.117 97.282 0)
       (effects (font (size 1.27 1.27)) (justify left))
     )
@@
   (symbol (lib_id "MCP25625-E_ML:MCP25625-E{slash}ML") (at 127.762 76.454 0) (unit 1)
     (in_bom yes) (on_board yes) (fields_autoplaced)
-    (property "Reference" "U?" (id 0) (at 160.1217 60.0542 0)
+    (property "Reference" "U3" (id 0) (at 160.1217 60.0542 0)
       (effects (font (size 1.27 1.27)) (justify left))
     )
@@
   (symbol (lib_id "Device:C") (at 222.758 69.088 180) (unit 1)
     (in_bom yes) (on_board yes)
-    (property "Reference" "C?" (id 0) (at 229.743 70.358 0)
+    (property "Reference" "C26" (id 0) (at 229.743 70.358 0)
       (effects (font (size 1.27 1.27)) (justify left))
     )
@@
   (symbol (lib_id "Device:C") (at 189.992 90.424 180) (unit 1)
     (in_bom yes) (on_board yes)
-    (property "Reference" "C?" (id 0) (at 186.944 91.694 0)
+    (property "Reference" "C24" (id 0) (at 186.944 91.694 0)
       (effects (font (size 1.27 1.27)) (justify left))
     )
@@
   (symbol (lib_id "Device:C") (at 212.598 79.248 180) (unit 1)
     (in_bom yes) (on_board yes)
-    (property "Reference" "C?" (id 0) (at 209.677 80.4164 0)
+    (property "Reference" "C25" (id 0) (at 209.677 80.4164 0)
       (effects (font (size 1.27 1.27)) (justify left))
     )
@@
   (symbol (lib_id "power:GND") (at 215.138 69.088 90) (unit 1)
     (in_bom yes) (on_board yes)
-    (property "Reference" "#PWR?" (id 0) (at 221.488 69.088 0)
+    (property "Reference" "#PWR0121" (id 0) (at 221.488 69.088 0)
       (effects (font (size 1.27 1.27)) hide)
     )
@@
   (symbol (lib_id "power:GND") (at 169.672 52.832 0) (unit 1)
     (in_bom yes) (on_board yes) (fields_autoplaced)
-    (property "Reference" "#PWR?" (id 0) (at 169.672 59.182 0)
+    (property "Reference" "#PWR0125" (id 0) (at 169.672 59.182 0)
       (effects (font (size 1.27 1.27)) hide)
     )
@@
   (symbol (lib_id "Device:R_Small") (at 107.188 73.406 0) (unit 1)
     (in_bom yes) (on_board yes)
-    (property "Reference" "R?" (id 0) (at 107.95 72.898 0)
+    (property "Reference" "R6" (id 0) (at 107.95 72.898 0)
       (effects (font (size 1.27 1.27)) (justify left))
     )
@@
   (symbol (lib_id "Device:C") (at 107.188 89.916 180) (unit 1)
     (in_bom yes) (on_board yes)
-    (property "Reference" "C?" (id 0) (at 104.14 91.186 0)
+    (property "Reference" "C23" (id 0) (at 104.14 91.186 0)
       (effects (font (size 1.27 1.27)) (justify left))
     )
@@
   (symbol (lib_id "power:GND") (at 107.188 96.012 0) (unit 1)
     (in_bom yes) (on_board yes) (fields_autoplaced)
-    (property "Reference" "#PWR?" (id 0) (at 107.188 102.362 0)
+    (property "Reference" "#PWR0124" (id 0) (at 107.188 102.362 0)
       (effects (font (size 1.27 1.27)) hide)
     )
@@
   (symbol (lib_id "power:GND") (at 180.848 124.968 0) (unit 1)
     (in_bom yes) (on_board yes) (fields_autoplaced)
-    (property "Reference" "#PWR?" (id 0) (at 180.848 131.318 0)
+    (property "Reference" "#PWR0123" (id 0) (at 180.848 131.318 0)
       (effects (font (size 1.27 1.27)) hide)
     )
@@
   (symbol (lib_id "power:GND") (at 210.058 69.088 270) (unit 1)
     (in_bom yes) (on_board yes)
-    (property "Reference" "#PWR?" (id 0) (at 203.708 69.088 0)
-      (effects (font (size 1.27 1.27)) hide)
-    )
+    (property "Reference" "#PWR0122" (id 0) (at 203.708 69.088 0)
+      (effects (font (size 1.27 1.27)) hide)
+    )
