File: CAN.kicad_sch (KiCad schematic)
At the start: 9 parts, among them U3 MCP25625-E/ML, Y1 16MHz

Commit message: steps added, before shorten
Parts:
- U3: footprint tuna-f1sh/jbr-kicad/QFN.pretty:QFN-28L -> QFN-28L
Connections:
- net GND: now also C25.1, C26.1
- net at C25.2, Y1.1: now also U3.20 (OSC2)
- no-connect marks 8 -> 6

Commit message: before removal of Nordic passive footprints
Parts:
- C23, C24, C25, C26: footprint MCU_Nordic_Accessory:C_0201 -> Capacitor_SMD:C_0201_0603Metric
- U3: footprint QFN-28L -> tuna-f1sh/jbr-kicad/QFN.pretty:QFN-28L
Changed lines of the file:
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@@
       (effects (font (size 1.27 1.27)) (justify left))
     )
-    (property "Footprint" "QFN-28L" (at 127.762 76.454 0)
+    (property "Footprint" "tuna-f1sh/jbr-kicad/QFN.pretty:QFN-28L" (at 127.762 76.454 0)
       (effects (font (size 1.27 1.27)) (justify bottom) hide)
     )
@@
       (effects (font (size 1.27 1.27)) (justify left))
     )
-    (property "Footprint" "MCU_Nordic_Accessory:C_0201" (at 221.7928 65.278 0)
+    (property "Footprint" "Capacitor_SMD:C_0201_0603Metric" (at 221.7928 65.278 0)
       (effects (font (size 1.27 1.27)) hide)
     )
@@
       (effects (font (size 1.27 1.27)) (justify left))
     )
-    (property "Footprint" "MCU_Nordic_Accessory:C_0201" (at 189.0268 86.614 0)
+    (property "Footprint" "Capacitor_SMD:C_0201_0603Metric" (at 189.0268 86.614 0)
       (effects (font (size 1.27 1.27)) hide)
     )
@@
       (effects (font (size 1.27 1.27)) (justify left))
     )
-    (property "Footprint" "MCU_Nordic_Accessory:C_0201" (at 211.6328 75.438 0)
+    (property "Footprint" "Capacitor_SMD:C_0201_0603Metric" (at 211.6328 75.438 0)
       (effects (font (size 1.27 1.27)) hide)
     )
@@
       (effects (font (size 1.27 1.27)) (justify left))
     )
-    (property "Footprint" "MCU_Nordic_Accessory:C_0201" (at 106.2228 86.106 0)
-      (effects (font (size 1.27 1.27)) hide)
-    )
+    (property "Footprint" "Capacitor_SMD:C_0201_0603Metric" (at 106.2228 86.106 0)
+      (effects (font (size 1.27 1.27)) hide)
+    )

Commit message: update BoM
Parts:
- U3: MFN (none) -> Microchip Technology; MPN (none) -> MCP25625-E/ML; SKU (none) -> MCP25625-E/ML-ND; Vendor (none) -> Digikey
Changed lines of the file:
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@@
       (effects (font (size 1.27 1.27)) hide)
     )
-    (property "MFN" "" (at 127.762 76.454 0)
+    (property "MFN" "Microchip Technology" (at 127.762 76.454 0)
       (effects (font (size 1.27 1.27)) hide)
     )
-    (property "MPN" "" (at 127.762 76.454 0)
+    (property "MPN" "MCP25625-E/ML" (at 127.762 76.454 0)
       (effects (font (size 1.27 1.27)) hide)
     )
-    (property "Description" "" (at 127.762 76.454 0)
+    (property "Description" "1/1 Transceiver CANbus 28-QFN (6x6)" (at 127.762 76.454 0)
       (effects (font (size 1.27 1.27)) hide)
     )
@@
       (effects (font (size 1.27 1.27)) hide)
     )
-    (property "Vendor" "" (at 127.762 76.454 0)
+    (property "Vendor" "Digikey" (at 127.762 76.454 0)
       (effects (font (size 1.27 1.27)) hide)
     )
-    (property "SKU" "" (at 127.762 76.454 0)
+    (property "SKU" "MCP25625-E/ML-ND" (at 127.762 76.454 0)
       (effects (font (size 1.27 1.27)) hide)
     )

Commit message: pre-production checks
Other:
- title: Spirit Logger -> CAN
Changed lines of the file:
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@@
   (paper "A4")
   (title_block
-    (title "Spirit Logger")
-    (date "2023-01-23")
+    (title "CAN")
+    (date "2023-02-28")
     (rev "0")
     (company "Specialized Europe GmbH")
+    (comment 1 "J.Whittington 2023")
   )
   (junction (at 180.848 104.394) (diameter 0) (color 0 0 0 0)
@@
       (effects (font (size 1.27 1.27)) (justify bottom) hide)
     )
-    (property "Datasheet" "" (at 127.762 76.454 0)
-      (effects (font (size 1.27 1.27)) hide)
-    )
+    (property "Datasheet" "https://ww1.microchip.com/downloads/aemDocuments/documents/OTH/ProductDocuments/DataSheets/MCP25625-CAN-Controller-Data-Sheet-20005282C.pdf" (at 127.762 76.454 0)
+      (effects (font (size 1.27 1.27)) hide)
+    )
