File: USB.kicad_sch (KiCad schematic)
At the start: 22 parts

Commit message: rename; annotate and import to pcb
Parts:
- U4: renamed from U?; value SN74LVC1G08DRYR -> SN74LVC1G00DRY2; symbol 74xGxx:74AHC1G08 -> 74xGxx:74AHC1G00; MPN SN74LVC1G08DRYR -> SN74LVC1G00DRY2; SKU 296-21815-1-ND -> 296-SN74LVC1G00DRY2CT-ND
- gave numbers to parts that had none: 11
Other:
- moved on the sheet: C27, C30, C31, C32, C33, C34, D1, FB1, FB2, FB3, J3, R55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
