File: USB.kicad_sch (KiCad schematic)
At the start: 22 parts, among them J3 USB_C_Receptacle, U4 SN74LVC1G00DRY2, U5 74CBTLV3245BQ

Commit message: drc updated for pcbway advanced; layout and tidy
Parts:
- J3: footprint Connector_USB:USB_C_Receptacle_GCT_USB4105-xx-A_16P_TopMnt_Horizontal -> Connector_USB:USB_C_Receptacle_Amphenol_12401610E4-2A
Changed lines of the file:
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@@
     (property "Reference" "J3" (id 0) (at 133.604 109.5334 0))
     (property "Value" "USB_C_Receptacle" (id 1) (at 133.604 112.0703 0))
-    (property "Footprint" "Connector_USB:USB_C_Receptacle_GCT_USB4105-xx-A_16P_TopMnt_Horizontal" (id 2) (at 137.414 141.1732 0)
+    (property "Footprint" "Connector_USB:USB_C_Receptacle_Amphenol_12401610E4-2A" (id 2) (at 137.414 141.1732 0)
       (effects (font (size 1.27 1.27)) hide)
     )
-    (property "Datasheet" "https://www.usb.org/sites/default/files/documents/usb_type-c.zip" (id 3) (at 137.414 141.1732 0)
+    (property "Datasheet" "" (id 3) (at 137.414 141.1732 0)
       (effects (font (size 1.27 1.27)) hide)
     )

Commit message: steps added, before shorten
Connections:
- net TX_N: now reaches J3.A3 (TX1-), TP9.1
- net TX_N: now also U5.3 (A2); no longer U5.2 (A1)
- net TX_P: now reaches J3.A2 (TX1+), TP10.1
- net TX_P: now also U5.2 (A1); no longer U5.3 (A2)

Commit message: before removal of Nordic passive footprints
Parts:
- C27, C30, C31, C32, C33: footprint MCU_Nordic_Accessory:C_0201 -> Capacitor_SMD:C_0201_0603Metric
- C34: footprint MCU_Nordic_Accessory:C_0603 -> Capacitor_SMD:C_0603_1608Metric
- D1: footprint MCU_Nordic_Accessory:SOT-143 -> Package_TO_SOT_SMD:SOT-143
- FB1, FB2, FB3: footprint MCU_Nordic_Accessory:FB_0603 -> Inductor_SMD:L_0603_1608Metric
Changed lines of the file:
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@@
       (effects (font (size 1.27 1.27)))
     )
-    (property "Footprint" "MCU_Nordic_Accessory:FB_0603" (at 150.114 62.4332 0)
+    (property "Footprint" "Inductor_SMD:L_0603_1608Metric" (at 150.114 62.4332 0)
       (effects (font (size 1.27 1.27)) hide)
     )
@@
       (effects (font (size 1.27 1.27)))
     )
-    (property "Footprint" "MCU_Nordic_Accessory:SOT-143" (at 168.91 97.9932 0)
+    (property "Footprint" "Package_TO_SOT_SMD:SOT-143" (at 168.91 97.9932 0)
       (effects (font (size 1.27 1.27)) hide)
     )
@@
       (effects (font (size 1.27 1.27)) (justify left))
     )
-    (property "Footprint" "MCU_Nordic_Accessory:C_0201" (at 158.6992 73.8632 0)
+    (property "Footprint" "Capacitor_SMD:C_0201_0603Metric" (at 158.6992 73.8632 0)
       (effects (font (size 1.27 1.27)) hide)
     )
@@
       (effects (font (size 1.27 1.27)) (justify left))
     )
-    (property "Footprint" "MCU_Nordic_Accessory:C_0201" (at 144.7292 73.8632 0)
+    (property "Footprint" "Capacitor_SMD:C_0201_0603Metric" (at 144.7292 73.8632 0)
       (effects (font (size 1.27 1.27)) hide)
     )
@@
       (effects (font (size 1.27 1.27)) (justify left))
     )
-    (property "Footprint" "MCU_Nordic_Accessory:C_0201" (at 236.728 138.938 0)
+    (property "Footprint" "Capacitor_SMD:C_0201_0603Metric" (at 236.728 138.938 0)
       (effects (font (size 1.27 1.27)) hide)
     )
@@
       (effects (font (size 1.27 1.27)))
     )
-    (property "Footprint" "MCU_Nordic_Accessory:FB_0603" (at 139.954 214.5792 0)
+    (property "Footprint" "Inductor_SMD:L_0603_1608Metric" (at 139.954 214.5792 0)
       (effects (font (size 1.27 1.27)) hide)
     )
@@
       (effects (font (size 1.27 1.27)))
     )
-    (property "Footprint" "MCU_Nordic_Accessory:FB_0603" (at 151.384 185.3692 0)
+    (property "Footprint" "Inductor_SMD:L_0603_1608Metric" (at 151.384 185.3692 0)
       (effects (font (size 1.27 1.27)) hide)
     )
@@
       (effects (font (size 1.27 1.27)) (justify left))
     )
-    (property "Footprint" "MCU_Nordic_Accessory:C_0201" (at 158.6992 89.1032 0)
+    (property "Footprint" "Capacitor_SMD:C_0201_0603Metric" (at 158.6992 89.1032 0)
       (effects (font (size 1.27 1.27)) hide)
     )
@@
       (effects (font (size 1.27 1.27)))
     )
-    (property "Footprint" "MCU_Nordic_Accessory:C_0201" (at 143.764 198.374 0)
+    (property "Footprint" "Capacitor_SMD:C_0201_0603Metric" (at 143.764 198.374 0)
       (effects (font (size 1.27 1.27)) hide)
     )
@@
       (effects (font (size 1.27 1.27)) (justify left))
     )
-    (property "Footprint" "MCU_Nordic_Accessory:C_0603" (at 144.7292 89.1032 0)
-      (effects (font (size 1.27 1.27)) hide)
-    )
+    (property "Footprint" "Capacitor_SMD:C_0603_1608Metric" (at 144.7292 89.1032 0)
+      (effects (font (size 1.27 1.27)) hide)
+    )

Commit message: update BoM
Parts:
- C27, C30, C31, C32, C33: Characteristics (none) -> X7R 6V
- C34: Characteristics (none) -> X5R 25V
- D1: Characteristics (none) -> TVS DIODE 5.5VWM SOT143B; MFN (none) -> Nexperia USA Inc.; MPN (none) -> PRTR5V0U2X,215; SKU (none) -> 1727-3884-1-ND; Vendor (none) -> Digikey
- FB1, FB2, FB3: Characteristics (none) -> 120R/0.55A; MFN (none) -> Laird-Signal Integrity Products; MPN (none) -> LI0603E151R-10; SKU (none) -> 240-2366-1-ND; Vendor (none) -> Digikey
- R55: Characteristics (none) -> 5%
- R7, R8: Characteristics 5% -> 1%
- U5: MFN (none) -> Nexperia USA Inc.; MPN (none) -> 74CBTLV3245BQ,115; SKU (none) -> 1727-6906-1-ND; Vendor (none) -> Digikey
Changed lines of the file:
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@@
+      (effects (font (size 1.27 1.27)) hide)
+    )
+    (property "Vendor" "Digikey" (at 248.666 161.4932 0)
+      (effects (font (size 1.27 1.27)) hide)
+    )
+    (property "Description" "Bus Switch 8 x 1:1 20-DHVQFN (4.5x2.5)" (at 248.666 161.4932 0)
+      (effects (font (size 1.27 1.27)) hide)
+    )
+    (property "MFN" "Nexperia USA Inc." (at 248.666 161.4932 0)
+      (effects (font (size 1.27 1.27)) hide)
+    )
+    (property "MPN" "74CBTLV3245BQ,115" (at 248.666 161.4932 0)
+      (effects (font (size 1.27 1.27)) hide)
+    )
+    (property "SKU" "1727-6906-1-ND" (at 248.666 161.4932 0)
       (effects (font (size 1.27 1.27)) hide)
     )
@@
       (effects (font (size 1.27 1.27)) hide)
     )
-    (property "Characteristics" "5%" (at 173.6344 128.7272 0)
+    (property "Characteristics" "1%" (at 173.6344 128.7272 0)
       (effects (font (size 1.27 1.27)) hide)
     )
@@
       (effects (font (size 1.27 1.27)) hide)
     )
+    (property "Characteristics" "120R/0.55A" (at 150.114 62.4332 0)
+      (effects (font (size 1.27 1.27)) hide)
+    )
+    (property "Description" "150 Ohms @ 100 MHz 1 Power, Signal Line Ferrite Bead 0603 (1608 Metric) 500mA 250mOhm" (at 150.114 62.4332 0)
+      (effects (font (size 1.27 1.27)) hide)
+    )
+    (property "MFN" "Laird-Signal Integrity Products" (at 150.114 62.4332 0)
+      (effects (font (size 1.27 1.27)) hide)
+    )
+    (property "MPN" "LI0603E151R-10" (at 150.114 62.4332 0)
+      (effects (font (size 1.27 1.27)) hide)
+    )
+    (property "SKU" "240-2366-1-ND" (at 150.114 62.4332 0)
+      (effects (font (size 1.27 1.27)) hide)
+    )
+    (property "Vendor" "Digikey" (at 150.114 62.4332 0)
+      (effects (font (size 1.27 1.27)) hide)
+    )
     (pin "1")
     (pin "2")
@@
     )
     (property "Datasheet" "https://assets.nexperia.com/documents/data-sheet/PRTR5V0U2X.pdf" (at 168.91 97.9932 0)
+      (effects (font (size 1.27 1.27)) hide)
+    )
+    (property "Description" "Clamp Ipp Tvs Diode Surface Mount SOT-143B" (at 170.434 97.9932 0)
+      (effects (font (size 1.27 1.27)) hide)
+    )
+    (property "MFN" "Nexperia USA Inc." (at 170.434 97.9932 0)
+      (effects (font (size 1.27 1.27)) hide)
+    )
+    (property "MPN" "PRTR5V0U2X,215" (at 170.434 97.9932 0)
+      (effects (font (size 1.27 1.27)) hide)
+    )
+    (property "SKU" "1727-3884-1-ND" (at 170.434 97.9932 0)
+      (effects (font (size 1.27 1.27)) hide)
+    )
+    (property "Vendor" "Digikey" (at 170.434 97.9932 0)
+      (effects (font (size 1.27 1.27)) hide)
+    )
+    (property "Characteristics" "TVS DIODE 5.5VWM SOT143B" (at 170.434 97.9932 0)
       (effects (font (size 1.27 1.27)) hide)
     )
@@
       (effects (font (size 1.27 1.27)) hide)
     )
+    (property "Characteristics" "5%" (at 139.954 205.6892 0)
+      (effects (font (size 1.27 1.27)) hide)
+    )
     (pin "1")
     (pin "2")
@@
       (effects (font (size 1.27 1.27)) hide)
     )
+    (property "Characteristics" "X7R 6V" (at 157.734 70.0532 0)
+      (effects (font (size 1.27 1.27)) hide)
+    )
     (pin "1")
     (pin "2")
@@
       (effects (font (size 1.27 1.27)) hide)
     )
-    (property "Characteristics" "5%" (at 168.3004 128.7272 0)
+    (property "Characteristics" "1%" (at 168.3004 128.7272 0)
       (effects (font (size 1.27 1.27)) hide)
     )
@@
       (effects (font (size 1.27 1.27)) hide)
     )
+    (property "Characteristics" "X7R 6V" (at 143.764 70.0532 0)
+      (effects (font (size 1.27 1.27)) hide)
+    )
     (pin "1")
     (pin "2")
@@
       (effects (font (size 1.27 1.27)) hide)
     )
+    (property "Characteristics" "X7R 6V" (at 240.538 137.9728 0)
+      (effects (font (size 1.27 1.27)) hide)
+    )
     (pin "1")
     (pin "2")
@@
     )
     (property "Datasheet" "~" (at 139.954 214.5792 0)
+      (effects (font (size 1.27 1.27)) hide)
+    )
+    (property "Characteristics" "120R/0.55A" (at 139.954 214.5792 0)
+      (effects (font (size 1.27 1.27)) hide)
+    )
+    (property "Description" "150 Ohms @ 100 MHz 1 Power, Signal Line Ferrite Bead 0603 (1608 Metric) 500mA 250mOhm" (at 139.954 214.5792 0)
+      (effects (font (size 1.27 1.27)) hide)
+    )
+    (property "MFN" "Laird-Signal Integrity Products" (at 139.954 214.5792 0)
+      (effects (font (size 1.27 1.27)) hide)
+    )
+    (property "MPN" "LI0603E151R-10" (at 139.954 214.5792 0)
+      (effects (font (size 1.27 1.27)) hide)
+    )
+    (property "SKU" "240-2366-1-ND" (at 139.954 214.5792 0)
+      (effects (font (size 1.27 1.27)) hide)
+    )
+    (property "Vendor" "Digikey" (at 139.954 214.5792 0)
       (effects (font (size 1.27 1.27)) hide)
     )
@@
       (effects (font (size 1.27 1.27)) hide)
     )
+    (property "Characteristics" "120R/0.55A" (at 151.384 185.3692 0)
+      (effects (font (size 1.27 1.27)) hide)
+    )
+    (property "Description" "150 Ohms @ 100 MHz 1 Power, Signal Line Ferrite Bead 0603 (1608 Metric) 500mA 250mOhm" (at 151.384 185.3692 0)
+      (effects (font (size 1.27 1.27)) hide)
+    )
+    (property "MFN" "Laird-Signal Integrity Products" (at 151.384 185.3692 0)
+      (effects (font (size 1.27 1.27)) hide)
+    )
+    (property "MPN" "LI0603E151R-10" (at 151.384 185.3692 0)
+      (effects (font (size 1.27 1.27)) hide)
+    )
+    (property "SKU" "240-2366-1-ND" (at 151.384 185.3692 0)
+      (effects (font (size 1.27 1.27)) hide)
+    )
+    (property "Vendor" "Digikey" (at 151.384 185.3692 0)
+      (effects (font (size 1.27 1.27)) hide)
+    )
     (pin "1")
     (pin "2")
@@
       (effects (font (size 1.27 1.27)) hide)
     )
-    (property "Datasheet" "" (at 137.414 141.1732 0)
+    (property "Datasheet" "https://media.digikey.com/pdf/Data%20Sheets/Amphenol%20PDFs/12401832E402A_Dwg_RevX1_04-25-17.pdf" (at 137.414 141.1732 0)
       (effects (font (size 1.27 1.27)) hide)
     )
@@
       (effects (font (size 1.27 1.27)) hide)
     )
+    (property "Characteristics" "X7R 6V" (at 157.734 85.2932 0)
+      (effects (font (size 1.27 1.27)) hide)
+    )
     (pin "1")
     (pin "2")
@@
       (effects (font (size 1.27 1.27)) hide)
     )
+    (property "Characteristics" "X7R 6V" (at 139.954 199.3392 0)
+      (effects (font (size 1.27 1.27)) hide)
+    )
     (pin "1")
     (pin "2")
@@
       (effects (font (size 1.27 1.27)) hide)
     )
+    (property "Characteristics" "X5R 25V" (at 143.764 85.2932 0)
+      (effects (font (size 1.27 1.27)) hide)
+    )

Commit message: pre-production checks
Other:
- title: Spirit Logger -> USB
Changed lines of the file:
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@@
   (paper "A3")
   (title_block
-    (title "Spirit Logger")
-    (date "2023-01-23")
+    (title "USB")
+    (date "2023-02-28")
     (rev "0")
     (company "Specialized Europe GmbH")
+    (comment 1 "J.Whittington 2023")
   )
   (junction (at 161.544 58.9788) (diameter 0) (color 0 0 0 0)

Commit message: makefile
Parts:
- J3: MFN (none) -> Amphenol ICC (Commercial Products); MPN (none) -> 12401610E4#2A; SKU (none) -> 12401610E4#2ACT-ND; Vendor (none) -> Digkey
Changed lines of the file:
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@@
+      (effects (font (size 1.27 1.27)) hide)
+    )
+    (property "Description" "USB-C (USB TYPE-C) USB 3.2 Gen 2 (USB 3.1 Gen 2, Superspeed + (USB 3.1)) Receptacle Connector 24 Position Surface Mount, Right Angle; Through Hole" (at 133.604 141.1732 0)
+      (effects (font (size 1.27 1.27)) hide)
+    )
+    (property "MFN" "Amphenol ICC (Commercial Products)" (at 133.604 141.1732 0)
+      (effects (font (size 1.27 1.27)) hide)
+    )
+    (property "MPN" "12401610E4#2A" (at 133.604 141.1732 0)
+      (effects (font (size 1.27 1.27)) hide)
+    )
+    (property "SKU" "12401610E4#2ACT-ND" (at 133.604 141.1732 0)
+      (effects (font (size 1.27 1.27)) hide)
+    )
+    (property "Vendor" "Digkey" (at 133.604 141.1732 0)
       (effects (font (size 1.27 1.27)) hide)
     )
