File: power.kicad_sch (KiCad schematic)
At the start: 12 parts

Commit message: rename; annotate and import to pcb
Parts:
- U7: renamed from U?; footprint Package_TO_SOT_SMD:SOT-363_SC-70-6 -> KiCad/Package_TO_SOT_SMD.pretty:SOT-363_SC-70-6
- gave numbers to parts that had none: 11
Changed lines of the file:
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@@
   (symbol (lib_id "power:GND") (at 164.9984 110.236 0) (unit 1)
     (in_bom yes) (on_board yes) (fields_autoplaced)
-    (property "Reference" "#PWR?" (id 0) (at 164.9984 116.586 0)
+    (property "Reference" "#PWR0138" (id 0) (at 164.9984 116.586 0)
       (effects (font (size 1.27 1.27)) hide)
     )
@@
   (symbol (lib_id "Device:C") (at 120.8024 138.684 0) (unit 1)
     (in_bom yes) (on_board yes)
-    (property "Reference" "C?" (id 0) (at 123.7234 137.5156 0)
+    (property "Reference" "C29" (id 0) (at 123.7234 137.5156 0)
       (effects (font (size 1.27 1.27)) (justify left))
     )
@@
   (symbol (lib_id "power:GND") (at 98.1964 120.269 0) (unit 1)
     (in_bom yes) (on_board yes) (fields_autoplaced)
-    (property "Reference" "#PWR?" (id 0) (at 98.1964 126.619 0)
+    (property "Reference" "#PWR0142" (id 0) (at 98.1964 126.619 0)
       (effects (font (size 1.27 1.27)) hide)
     )
@@
   (symbol (lib_id "power:GND") (at 162.4584 149.352 0) (unit 1)
     (in_bom yes) (on_board yes) (fields_autoplaced)
-    (property "Reference" "#PWR?" (id 0) (at 162.4584 155.702 0)
+    (property "Reference" "#PWR0139" (id 0) (at 162.4584 155.702 0)
       (effects (font (size 1.27 1.27)) hide)
     )
@@
   (symbol (lib_id "Connector:TestPoint_Small") (at 177.4444 126.365 0) (unit 1)
     (in_bom yes) (on_board yes)
-    (property "Reference" "TP?" (id 0) (at 177.419 124.4092 0)
+    (property "Reference" "TP13" (id 0) (at 177.419 124.4092 0)
       (effects (font (size 1.27 1.27)) (justify left))
     )
@@
   (symbol (lib_id "Device:R_Small") (at 103.6574 119.761 0) (unit 1)
     (in_bom yes) (on_board yes)
-    (property "Reference" "R?" (id 0) (at 104.4194 119.253 0)
+    (property "Reference" "R11" (id 0) (at 104.4194 119.253 0)
       (effects (font (size 1.27 1.27)) (justify left))
     )
@@
   (symbol (lib_id "Device:C") (at 167.4114 132.207 0) (unit 1)
     (in_bom yes) (on_board yes)
-    (property "Reference" "C?" (id 0) (at 170.3324 131.0386 0)
+    (property "Reference" "C35" (id 0) (at 170.3324 131.0386 0)
       (effects (font (size 1.27 1.27)) (justify left))
     )
@@
   (symbol (lib_id "LMZ21700SILR:LMZ21700SILR") (at 142.3924 123.825 0) (unit 1)
     (in_bom yes) (on_board yes) (fields_autoplaced)
-    (property "Reference" "U?" (id 0) (at 142.3924 102.2672 0))
+    (property "Reference" "U6" (id 0) (at 142.3924 102.2672 0))
     (property "Value" "LMZ21700SILR" (id 1) (at 142.3924 104.8041 0))
     (property "Footprint" "tunaf1sh/snapeda.pretty:CONV_TPS82140SILR" (id 2) (at 142.3924 123.825 0)
@@
   (symbol (lib_id "power:GND") (at 65.3796 110.6932 0) (unit 1)
     (in_bom yes) (on_board yes)
-    (property "Reference" "#PWR?" (id 0) (at 65.3796 110.6932 0)
+    (property "Reference" "#PWR0141" (id 0) (at 65.3796 110.6932 0)
       (effects (font (size 0.762 0.762)) hide)
     )
@@
   (symbol (lib_id "Diode:MBR0540") (at 86.8934 101.219 90) (unit 1)
     (in_bom yes) (on_board yes)
-    (property "Reference" "D?" (id 0) (at 88.9254 100.0506 90)
+    (property "Reference" "D4" (id 0) (at 88.9254 100.0506 90)
       (effects (font (size 1.27 1.27)) (justify right))
     )
@@
   (symbol (lib_id "Power_Management:SiP32432DR3") (at 284.8864 120.8532 0) (unit 1)
     (in_bom yes) (on_board yes) (fields_autoplaced)
-    (property "Reference" "U?" (id 0) (at 284.8864 112.0734 0))
+    (property "Reference" "U7" (id 0) (at 284.8864 112.0734 0))
     (property "Value" "SiP32432DR3" (id 1) (at 284.8864 114.6103 0))
-    (property "Footprint" "Package_TO_SOT_SMD:SOT-363_SC-70-6" (id 2) (at 284.8864 109.4232 0)
+    (property "Footprint" "KiCad/Package_TO_SOT_SMD.pretty:SOT-363_SC-70-6" (id 2) (at 284.8864 109.4232 0)
       (effects (font (size 1.27 1.27)) hide)
     )
@@
   (symbol (lib_id "Device:R_Small") (at 171.0944 122.555 0) (unit 1)
     (in_bom yes) (on_board yes)
-    (property "Reference" "R?" (id 0) (at 171.8564 122.047 0)
+    (property "Reference" "R13" (id 0) (at 171.8564 122.047 0)
       (effects (font (size 1.27 1.27)) (justify left))
     )
@@
   (symbol (lib_id "Device:C") (at 89.9414 113.284 0) (unit 1)
     (in_bom yes) (on_board yes)
-    (property "Reference" "C?" (id 0) (at 92.8624 112.1156 0)
+    (property "Reference" "C28" (id 0) (at 92.8624 112.1156 0)
       (effects (font (size 1.27 1.27)) (justify left))
     )
@@
   (symbol (lib_id "Device:R_Small") (at 65.3796 98.7552 0) (unit 1)
     (in_bom yes) (on_board yes)
-    (property "Reference" "R?" (id 0) (at 66.1416 98.2472 0)
+    (property "Reference" "R9" (id 0) (at 66.1416 98.2472 0)
       (effects (font (size 1.27 1.27)) (justify left))
     )
@@
   (symbol (lib_id "power:GND") (at 284.8864 129.9972 0) (unit 1)
     (in_bom yes) (on_board yes) (fields_autoplaced)
-    (property "Reference" "#PWR?" (id 0) (at 284.8864 136.3472 0)
+    (property "Reference" "#PWR0140" (id 0) (at 284.8864 136.3472 0)
       (effects (font (size 1.27 1.27)) hide)
     )
@@
   (symbol (lib_id "Device:R_Small") (at 65.3796 106.6292 0) (unit 1)
     (in_bom yes) (on_board yes)
-    (property "Reference" "R?" (id 0) (at 66.1416 106.1212 0)
+    (property "Reference" "R10" (id 0) (at 66.1416 106.1212 0)
       (effects (font (size 1.27 1.27)) (justify left))
     )
@@
   (symbol (lib_id "Device:R_Small") (at 103.6574 127.889 0) (unit 1)
     (in_bom yes) (on_board yes)
-    (property "Reference" "R?" (id 0) (at 104.4194 127.381 0)
-      (effects (font (size 1.27 1.27)) (justify left))
-    )
+    (property "Reference" "R12" (id 0) (at 104.4194 127.381 0)
+      (effects (font (size 1.27 1.27)) (justify left))
+    )
