File: power.kicad_sch (KiCad schematic)
At the start: 13 parts, among them U6 LMZ21700SILR, U7 SiP32432DR3

Commit message: steps added, before shorten
Parts:
- U6: footprint tuna-f1sh/jbr-kicad/SnapEDA.pretty:CONV_TPS82140SILR -> tuna-f1sh/jbr-kicad/SnapEDA.pretty:Texas_Instruments-SIL0008E-0-0-MFG
Connections:
- net VOUT is gone; now on net DCDC_VOUT: R12.2, U6.6 (VOS)
- net GND: no longer U6.11 (PAD@3), U6.12 (PAD@4)

Commit message: before removal of Nordic passive footprints
Parts:
- C29: footprint MCU_Nordic_Accessory:C_0201 -> Capacitor_SMD:C_0201_0603Metric
Changed lines of the file:
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@@
       (effects (font (size 1.27 1.27)) (justify left))
     )
-    (property "Footprint" "MCU_Nordic_Accessory:C_0201" (at 121.7676 142.494 0)
+    (property "Footprint" "Capacitor_SMD:C_0201_0603Metric" (at 121.7676 142.494 0)
       (effects (font (size 1.27 1.27)) hide)
     )

Commit message: update BoM
Parts:
- U7: MFN (none) -> Vishay Siliconix; MPN (none) -> SIP32432DR3-T1GE3; SKU (none) -> SIP32432DR3-T1GE3CT-ND; Vendor (none) -> Digikey
Changed lines of the file:
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@@
+      (effects (font (size 1.27 1.27)) hide)
+    )
+    (property "Description" "IC PWR SWITCH P-CHAN 1:1 SC70-6" (at 284.8864 120.8532 0)
+      (effects (font (size 1.27 1.27)) hide)
+    )
+    (property "MFN" "Vishay Siliconix" (at 284.8864 120.8532 0)
+      (effects (font (size 1.27 1.27)) hide)
+    )
+    (property "MPN" "SIP32432DR3-T1GE3" (at 284.8864 120.8532 0)
+      (effects (font (size 1.27 1.27)) hide)
+    )
+    (property "SKU" "SIP32432DR3-T1GE3CT-ND" (at 284.8864 120.8532 0)
+      (effects (font (size 1.27 1.27)) hide)
+    )
+    (property "Vendor" "Digikey" (at 284.8864 120.8532 0)
       (effects (font (size 1.27 1.27)) hide)
     )

Commit message: pre-production checks
Parts:
- R12: value 240k -> 232k
Other:
- note added: "12V (17V max) -> 5.45V DCDC buck RFBT = RFBB x (VOUT/ 0.8 - 1)"
- note removed: "12V (17V max) -> 5.6V DCDC buck"
- title: Spirit Logger -> Power
Changed lines of the file:
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@@
   (paper "A3")
   (title_block
-    (title "Spirit Logger")
-    (date "2023-01-23")
+    (title "Power")
+    (date "2023-02-28")
     (rev "0")
     (company "Specialized Europe GmbH")
+    (comment 1 "J.Whittington 2023")
   )
   (junction (at 103.6828 123.8504) (diameter 0) (color 0 0 0 0)
@@
     )
   )
-  (text "12V (17V max) -> 5.6V DCDC buck" (at 124.8156 91.2368 0)
+  (text "12V (17V max) -> 5.45V DCDC buck\nRFBT = RFBB x (VOUT/ 0.8 - 1)"
+    (at 124.8156 91.2368 0)
     (effects (font (size 1.27 1.27)) (justify left bottom))
   )
@@
       (effects (font (size 1.27 1.27)) hide)
     )
-    (property "Datasheet" "http://www.vishay.com.hk/docs/66597/sip32431.pdf" (at 284.8864 120.8532 0)
+    (property "Datasheet" "https://www.vishay.com/docs/66597/sip32431.pdf" (at 284.8864 120.8532 0)
       (effects (font (size 1.27 1.27)) hide)
     )
@@
     )
     (property "Vendor" "Digikey" (at 284.8864 120.8532 0)
+      (effects (font (size 1.27 1.27)) hide)
+    )
+    (property "Notes" "" (at 284.8864 120.8532 0)
+      (effects (font (size 1.27 1.27)) hide)
+    )
+    (property "Config" "" (at 284.8864 120.8532 0)
+      (effects (font (size 1.27 1.27)) hide)
+    )
+    (property "Characteristics" "" (at 284.8864 120.8532 0)
       (effects (font (size 1.27 1.27)) hide)
     )
@@
       (effects (font (size 1.27 1.27)) (justify left))
     )
-    (property "Value" "240k" (at 104.4448 128.9304 0)
+    (property "Value" "232k" (at 104.4448 128.9304 0)
       (effects (font (size 1.27 1.27)) (justify left))
     )
@@
       (effects (font (size 1.27 1.27)) hide)
     )
+    (property "MFN" "" (at 103.6828 127.9144 0)
+      (effects (font (size 1.27 1.27)) hide)
+    )
+    (property "MPN" "" (at 103.6828 127.9144 0)
+      (effects (font (size 1.27 1.27)) hide)
+    )
+    (property "Description" "" (at 103.6828 127.9144 0)
+      (effects (font (size 1.27 1.27)) hide)
+    )
+    (property "Notes" "" (at 103.6828 127.9144 0)
+      (effects (font (size 1.27 1.27)) hide)
+    )
+    (property "Config" "" (at 103.6828 127.9144 0)
+      (effects (font (size 1.27 1.27)) hide)
+    )
+    (property "Vendor" "" (at 103.6828 127.9144 0)
+      (effects (font (size 1.27 1.27)) hide)
+    )
+    (property "SKU" "" (at 103.6828 127.9144 0)
+      (effects (font (size 1.27 1.27)) hide)
+    )

Commit message: makefile
Parts:
- D4, D6: Characteristics DIODE SCHOTTKY 40V 500MA SOD123 -> > 15 V forward and low drop; MFN ON Semiconductor -> Panjit International Inc.; MPN MBR0540T3G -> SS0520_R1_00001; SKU MBR0540T3GOSCT-ND -> 3757-SS0520_R1_00001CT-ND
- R9: value 50k -> 49.9k
Changed lines of the file:
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@@
       (effects (font (size 1.27 1.27)) hide)
     )
-    (property "Characteristics" "DIODE SCHOTTKY 40V 500MA SOD123" (at 86.9188 101.2444 0)
-      (effects (font (size 1.27 1.27)) hide)
-    )
-    (property "Description" "Diode Schottky 40V 500mA Surface Mount SOD-123" (at 86.9188 101.2444 0)
-      (effects (font (size 1.27 1.27)) hide)
-    )
-    (property "MFN" "ON Semiconductor" (at 86.9188 101.2444 0)
-      (effects (font (size 1.27 1.27)) hide)
-    )
-    (property "MPN" "MBR0540T3G" (at 86.9188 101.2444 0)
-      (effects (font (size 1.27 1.27)) hide)
-    )
-    (property "SKU" "MBR0540T3GOSCT-ND" (at 86.9188 101.2444 0)
+    (property "Characteristics" "> 15 V forward and low drop" (at 86.9188 101.2444 0)
+      (effects (font (size 1.27 1.27)) hide)
+    )
+    (property "Description" "Diode 20 V 500mA Surface Mount SOD-123" (at 86.9188 101.2444 0)
+      (effects (font (size 1.27 1.27)) hide)
+    )
+    (property "MFN" "Panjit International Inc." (at 86.9188 101.2444 0)
+      (effects (font (size 1.27 1.27)) hide)
+    )
+    (property "MPN" "SS0520_R1_00001" (at 86.9188 101.2444 0)
+      (effects (font (size 1.27 1.27)) hide)
+    )
+    (property "SKU" "3757-SS0520_R1_00001CT-ND" (at 86.9188 101.2444 0)
       (effects (font (size 1.27 1.27)) hide)
     )
@@
       (effects (font (size 1.27 1.27)) (justify left))
     )
-    (property "Value" "50k" (at 66.1416 99.7712 0)
+    (property "Value" "49.9k" (at 66.1416 99.7712 0)
       (effects (font (size 1.27 1.27)) (justify left))
     )
@@
     )
     (property "Characteristics" "5%" (at 65.3796 98.7552 0)
+      (effects (font (size 1.27 1.27)) hide)
+    )
+    (property "MFN" "" (at 65.3796 98.7552 0)
+      (effects (font (size 1.27 1.27)) hide)
+    )
+    (property "MPN" "" (at 65.3796 98.7552 0)
+      (effects (font (size 1.27 1.27)) hide)
+    )
+    (property "Description" "" (at 65.3796 98.7552 0)
+      (effects (font (size 1.27 1.27)) hide)
+    )
+    (property "Notes" "" (at 65.3796 98.7552 0)
+      (effects (font (size 1.27 1.27)) hide)
+    )
+    (property "Config" "" (at 65.3796 98.7552 0)
+      (effects (font (size 1.27 1.27)) hide)
+    )
+    (property "Vendor" "" (at 65.3796 98.7552 0)
+      (effects (font (size 1.27 1.27)) hide)
+    )
+    (property "SKU" "" (at 65.3796 98.7552 0)
       (effects (font (size 1.27 1.27)) hide)
     )
@@
       (effects (font (size 1.27 1.27)) hide)
     )
-    (property "Characteristics" "DIODE SCHOTTKY 40V 500MA SOD123" (at 284.8864 143.256 0)
-      (effects (font (size 1.27 1.27)) hide)
-    )
-    (property "Description" "Diode Schottky 40V 500mA Surface Mount SOD-123" (at 284.8864 143.256 0)
-      (effects (font (size 1.27 1.27)) hide)
-    )
-    (property "MFN" "ON Semiconductor" (at 284.8864 143.256 0)
-      (effects (font (size 1.27 1.27)) hide)
-    )
-    (property "MPN" "MBR0540T3G" (at 284.8864 143.256 0)
-      (effects (font (size 1.27 1.27)) hide)
-    )
-    (property "SKU" "MBR0540T3GOSCT-ND" (at 284.8864 143.256 0)
-      (effects (font (size 1.27 1.27)) hide)
-    )
+    (property "Characteristics" "> 15 V forward and low drop" (at 284.8864 143.256 0)
+      (effects (font (size 1.27 1.27)) hide)
+    )
+    (property "Description" "Diode 20 V 500mA Surface Mount SOD-123" (at 284.8864 143.256 0)
+      (effects (font (size 1.27 1.27)) hide)
+    )
+    (property "MFN" "Panjit International Inc." (at 284.8864 143.256 0)
+      (effects (font (size 1.27 1.27)) hide)
+    )
+    (property "MPN" "SS0520_R1_00001" (at 284.8864 143.256 0)
+      (effects (font (size 1.27 1.27)) hide)
+    )
+    (property "SKU" "3757-SS0520_R1_00001CT-ND" (at 284.8864 143.256 0)
+      (effects (font (size 1.27 1.27)) hide)
+    )
