File: sensors.kicad_sch (KiCad schematic)
At the start: 15 parts

Commit message: rename; annotate and import to pcb
Parts:
- U8: renamed from U?; footprint KiCad/Package_LGA:LGA-14_3x2.5mm_P0.5mm_LayoutBorder3x4y -> KiCad/Package_LGA.pretty:LGA-14_3x2.5mm_P0.5mm_LayoutBorder3x4y
- gave numbers to parts that had none: 14
Changed lines of the file:
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@@
   (symbol (lib_id "power:GND") (at 226.3648 100.6348 0) (unit 1)
     (in_bom yes) (on_board yes)
-    (property "Reference" "#PWR?" (id 0) (at 226.3648 100.6348 0)
+    (property "Reference" "#PWR0147" (id 0) (at 226.3648 100.6348 0)
       (effects (font (size 0.762 0.762)) hide)
     )
@@
   (symbol (lib_id "Device:R_Small") (at 244.3988 96.5708 0) (unit 1)
     (in_bom yes) (on_board yes)
-    (property "Reference" "R?" (id 0) (at 245.1608 96.0628 0)
+    (property "Reference" "R20" (id 0) (at 245.1608 96.0628 0)
       (effects (font (size 1.27 1.27)) (justify left))
     )
@@
   (symbol (lib_id "Device:C") (at 54.9656 81.026 180) (unit 1)
     (in_bom yes) (on_board yes)
-    (property "Reference" "C?" (id 0) (at 51.9176 82.296 0)
+    (property "Reference" "C37" (id 0) (at 51.9176 82.296 0)
       (effects (font (size 1.27 1.27)) (justify left))
     )
@@
   (symbol (lib_id "Device:D_Zener") (at 188.976 99.1616 270) (unit 1)
     (in_bom yes) (on_board yes)
-    (property "Reference" "D?" (id 0) (at 190.9826 97.9932 90)
+    (property "Reference" "D5" (id 0) (at 190.9826 97.9932 90)
       (effects (font (size 1.27 1.27)) (justify left))
     )
@@
   (symbol (lib_id "Device:R_Small") (at 179.324 100.1776 0) (unit 1)
     (in_bom yes) (on_board yes)
-    (property "Reference" "R?" (id 0) (at 180.086 99.6696 0)
+    (property "Reference" "R15" (id 0) (at 180.086 99.6696 0)
       (effects (font (size 1.27 1.27)) (justify left))
     )
@@
   (symbol (lib_id "Connector:TestPoint_Small") (at 244.3988 83.9724 0) (unit 1)
     (in_bom yes) (on_board yes)
-    (property "Reference" "TP?" (id 0) (at 242.6462 82.4484 0)
+    (property "Reference" "TP16" (id 0) (at 242.6462 82.4484 0)
       (effects (font (size 1.27 1.27)) (justify left))
     )
@@
   (symbol (lib_id "power:GND") (at 244.3988 100.6348 0) (unit 1)
     (in_bom yes) (on_board yes)
-    (property "Reference" "#PWR?" (id 0) (at 244.3988 100.6348 0)
+    (property "Reference" "#PWR0148" (id 0) (at 244.3988 100.6348 0)
       (effects (font (size 0.762 0.762)) hide)
     )
@@
   (symbol (lib_id "power:VDD") (at 91.3892 72.9488 0) (unit 1)
     (in_bom yes) (on_board yes) (fields_autoplaced)
-    (property "Reference" "#PWR?" (id 0) (at 91.3892 76.7588 0)
+    (property "Reference" "#PWR0143" (id 0) (at 91.3892 76.7588 0)
       (effects (font (size 1.27 1.27)) hide)
     )
@@
   (symbol (lib_name "GND_1") (lib_id "power:GND") (at 54.9656 88.0364 0) (unit 1)
     (in_bom yes) (on_board yes) (fields_autoplaced)
-    (property "Reference" "#PWR?" (id 0) (at 54.9656 94.3864 0)
+    (property "Reference" "#PWR0144" (id 0) (at 54.9656 94.3864 0)
       (effects (font (size 1.27 1.27)) hide)
     )
@@
   (symbol (lib_id "Device:R_Small") (at 169.926 85.4456 0) (mirror x) (unit 1)
     (in_bom yes) (on_board yes)
-    (property "Reference" "R?" (id 0) (at 170.688 85.9536 0)
+    (property "Reference" "R14" (id 0) (at 170.688 85.9536 0)
       (effects (font (size 1.27 1.27)) (justify left))
     )
@@
   (symbol (lib_id "power:GND") (at 169.926 105.5116 0) (unit 1)
     (in_bom yes) (on_board yes)
-    (property "Reference" "#PWR?" (id 0) (at 169.926 105.5116 0)
+    (property "Reference" "#PWR0146" (id 0) (at 169.926 105.5116 0)
       (effects (font (size 0.762 0.762)) hide)
     )
@@
   (symbol (lib_id "Device:R_Small") (at 226.3648 88.6968 0) (unit 1)
     (in_bom yes) (on_board yes)
-    (property "Reference" "R?" (id 0) (at 227.1268 88.1888 0)
+    (property "Reference" "R17" (id 0) (at 227.1268 88.1888 0)
       (effects (font (size 1.27 1.27)) (justify left))
     )
@@
   (symbol (lib_id "Device:R_Small") (at 195.326 95.3516 270) (mirror x) (unit 1)
     (in_bom yes) (on_board yes)
-    (property "Reference" "R?" (id 0) (at 195.834 94.5896 0)
+    (property "Reference" "R16" (id 0) (at 195.834 94.5896 0)
       (effects (font (size 1.27 1.27)) (justify left))
     )
@@
   (symbol (lib_id "Connector:TestPoint_Small") (at 226.3648 83.8708 0) (unit 1)
     (in_bom yes) (on_board yes)
-    (property "Reference" "TP?" (id 0) (at 224.6122 82.3722 0)
+    (property "Reference" "TP15" (id 0) (at 224.6122 82.3722 0)
       (effects (font (size 1.27 1.27)) (justify left))
     )
@@
   (symbol (lib_name "GND_1") (lib_id "power:GND") (at 91.3892 113.3348 0) (unit 1)
     (in_bom yes) (on_board yes) (fields_autoplaced)
-    (property "Reference" "#PWR?" (id 0) (at 91.3892 119.6848 0)
+    (property "Reference" "#PWR0145" (id 0) (at 91.3892 119.6848 0)
       (effects (font (size 1.27 1.27)) hide)
     )
@@
   (symbol (lib_id "Device:C") (at 42.1132 81.026 180) (unit 1)
     (in_bom yes) (on_board yes)
-    (property "Reference" "C?" (id 0) (at 39.0652 82.296 0)
+    (property "Reference" "C36" (id 0) (at 39.0652 82.296 0)
       (effects (font (size 1.27 1.27)) (justify left))
     )
@@
   (symbol (lib_id "Device:R_Small") (at 244.3988 88.6968 0) (unit 1)
     (in_bom yes) (on_board yes)
-    (property "Reference" "R?" (id 0) (at 245.1608 88.1888 0)
+    (property "Reference" "R19" (id 0) (at 245.1608 88.1888 0)
       (effects (font (size 1.27 1.27)) (justify left))
     )
@@
   (symbol (lib_id "Device:R_Small") (at 226.3648 96.5708 0) (unit 1)
     (in_bom yes) (on_board yes)
-    (property "Reference" "R?" (id 0) (at 227.1268 96.0628 0)
+    (property "Reference" "R18" (id 0) (at 227.1268 96.0628 0)
       (effects (font (size 1.27 1.27)) (justify left))
     )
@@
   (symbol (lib_id "Transistor_FET:BSS123") (at 172.466 95.3516 0) (mirror y) (unit 1)
     (in_bom yes) (on_board yes)
-    (property "Reference" "Q?" (id 0) (at 167.2844 94.1832 0)
+    (property "Reference" "Q1" (id 0) (at 167.2844 94.1832 0)
       (effects (font (size 1.27 1.27)) (justify left))
     )
@@
   (symbol (lib_id "Connector:TestPoint_Small") (at 198.882 95.3516 270) (unit 1)
     (in_bom yes) (on_board yes)
-    (property "Reference" "TP?" (id 0) (at 199.8726 95.377 90)
+    (property "Reference" "TP14" (id 0) (at 199.8726 95.377 90)
       (effects (font (size 1.27 1.27)) (justify left))
     )
@@
   (symbol (lib_id "Sensor_Motion:LSM6DSL") (at 88.8492 93.218 0) (unit 1)
     (in_bom yes) (on_board yes) (fields_autoplaced)
-    (property "Reference" "U?" (id 0) (at 106.5937 79.8915 0))
+    (property "Reference" "U8" (id 0) (at 106.5937 79.8915 0))
     (property "Value" "LSM6DSL" (id 1) (at 106.5937 82.4284 0))
-    (property "Footprint" "KiCad/Package_LGA:LGA-14_3x2.5mm_P0.5mm_LayoutBorder3x4y" (id 2) (at 78.6892 110.998 0)
+    (property "Footprint" "KiCad/Package_LGA.pretty:LGA-14_3x2.5mm_P0.5mm_LayoutBorder3x4y" (id 2) (at 78.6892 110.998 0)
       (effects (font (size 1.27 1.27)) (justify left) hide)
     )
