File: sensors.kicad_sch (KiCad schematic)
At the start: 15 parts, among them Q1 BSS123, U8 LSM6DSL

Commit message: before removal of Nordic passive footprints
Parts:
- C36, C37: footprint MCU_Nordic_Accessory:C_0201 -> Capacitor_SMD:C_0201_0603Metric
Changed lines of the file:
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@@
       (effects (font (size 1.27 1.27)) (justify left))
     )
-    (property "Footprint" "MCU_Nordic_Accessory:C_0201" (at 54.0004 77.216 0)
+    (property "Footprint" "Capacitor_SMD:C_0201_0603Metric" (at 54.0004 77.216 0)
       (effects (font (size 1.27 1.27)) hide)
     )
@@
       (effects (font (size 1.27 1.27)) (justify left))
     )
-    (property "Footprint" "MCU_Nordic_Accessory:C_0201" (at 41.148 77.216 0)
-      (effects (font (size 1.27 1.27)) hide)
-    )
+    (property "Footprint" "Capacitor_SMD:C_0201_0603Metric" (at 41.148 77.216 0)
+      (effects (font (size 1.27 1.27)) hide)
+    )

Commit message: update BoM
Parts:
- R15, R17, R19: Characteristics 5% -> 1%
- U8: MFN (none) -> STMicroelectronics; MPN (none) -> LSM6DSLTR; SKU (none) -> 497-16705-1-ND; Vendor (none) -> Digikey
Changed lines of the file:
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@@
       (effects (font (size 1.27 1.27)) hide)
     )
-    (property "Characteristics" "5%" (at 179.324 100.1776 0)
+    (property "Characteristics" "1%" (at 179.324 100.1776 0)
       (effects (font (size 1.27 1.27)) hide)
     )
@@
       (effects (font (size 1.27 1.27)) hide)
     )
-    (property "Characteristics" "5%" (at 226.3648 88.6968 0)
+    (property "Characteristics" "1%" (at 226.3648 88.6968 0)
       (effects (font (size 1.27 1.27)) hide)
     )
@@
       (effects (font (size 1.27 1.27)) hide)
     )
-    (property "Characteristics" "5%" (at 244.3988 88.6968 0)
+    (property "Characteristics" "1%" (at 244.3988 88.6968 0)
       (effects (font (size 1.27 1.27)) hide)
     )
@@
       (effects (font (size 1.27 1.27)) hide)
     )
+    (property "Description" "Accelerometer, Gyroscope, Temperature, 6 Axis Sensor I²C, SPI Output" (at 88.8492 93.218 0)
+      (effects (font (size 1.27 1.27)) hide)
+    )
+    (property "MFN" "STMicroelectronics" (at 88.8492 93.218 0)
+      (effects (font (size 1.27 1.27)) hide)
+    )
+    (property "MPN" "LSM6DSLTR" (at 88.8492 93.218 0)
+      (effects (font (size 1.27 1.27)) hide)
+    )
+    (property "SKU" "497-16705-1-ND" (at 88.8492 93.218 0)
+      (effects (font (size 1.27 1.27)) hide)
+    )
+    (property "Vendor" "Digikey" (at 88.8492 93.218 0)
+      (effects (font (size 1.27 1.27)) hide)
+    )

Commit message: pre-production checks
Other:
- company: (none) -> Specialized Europe GmbH
- title: (none) -> Sensors
Changed lines of the file:
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@@
 (kicad_sch (version 20230121) (generator eeschema)
   (paper "A4")
+  (title_block
+    (title "Sensors")
+    (date "2023-02-28")
+    (rev "0")
+    (company "Specialized Europe GmbH")
+    (comment 1 "J.Whittington 2023")
+  )
   (junction (at 244.3988 92.7608) (diameter 0) (color 0 0 0 0)
   )
