File: spirit_logger_hardware.kicad_pcb (KiCad board)
At the start: 4 copper layers, 75 x 40 mm, 86 parts, among them P1 Conn_01x22, P2 Conn_01x22, P3 Conn_01x07, P4 Conn_01x06, SW1 SW_Push, SW2 SW_Push, U1 nRF5340-QKAA, U2 MX25R6435F, U4 SHTC3, X1 Crystal_GND24, X2 Crystal

Commit message: rename; annotate and import to pcb
Parts:
- removed H1, H2: MountingHole_Pad, MCU_Nordic_Accessory:MountingHole_2.5mm_Plated
- removed H3, H4: MountingHole, MCU_Nordic_Accessory:MountingHole_2.5mm
- removed P1, P2: Conn_01x22, MCU_Nordic_Accessory:PinHeader_1x022_P2.54mm_Vertical
- removed P3: Conn_01x07, MCU_Nordic_Accessory:PinHeader_1x07_P2.54mm_Vertical
- removed P4: Conn_01x06, MCU_Nordic_Accessory:PinHeader_1x06_P2.54mm_Vertical
- removed R53, R54: 0, MCU_Nordic_Accessory:R_0201
- removed SB0, SB1, SB10, SB11, SB12, SB13, SB14, SB15, SB17, SB2, SB3, SB4, SB5, SB6, SB7, SB8, SB9: DNI, MCU_Nordic_Accessory:SB_PAD_SHORT
- removed SW1, SW2: SW_Push, Button_Switch_SMD:Panasonic_EVQPUK_EVQPUB
- removed USB1: USB_B_Micro, Connector_USB:USB_Micro-B_Amphenol_10103594-0001LF_Horizontal
- added C23: 100nF, KiCad/Capacitor_SMD.pretty:C_0402_1005Metric_Pad0.74x0.62mm_HandSolder, F.Cu at (54.0, 27.6)
- added C24: 100nF, KiCad/Capacitor_SMD.pretty:C_0402_1005Metric_Pad0.74x0.62mm_HandSolder, F.Cu at (44.2, 35.4)
- added C25: 8pF, KiCad/Capacitor_SMD.pretty:C_0603_1608Metric, F.Cu at (49.1, 32.4)
- added C26: 8pF, KiCad/Capacitor_SMD.pretty:C_0603_1608Metric, F.Cu at (40.6, 35.6)
- added C27: 100nF, MCU_Nordic_Accessory:C_0201, F.Cu at (21.7, 37.4)
- added C28: 22u, KiCad/Capacitor_SMD.pretty:C_0805_2012Metric, F.Cu at (66.9, 21.5)
- added C29: 3.3n, KiCad/Capacitor_SMD.pretty:C_0402_1005Metric, F.Cu at (70.6, 23.0)
- added C35: 22u, KiCad/Capacitor_SMD.pretty:C_0805_2012Metric, F.Cu at (62.2, 26.1)
- added C36: 100nF, KiCad/Capacitor_SMD.pretty:C_0402_1005Metric_Pad0.74x0.62mm_HandSolder, F.Cu at (52.5, 15.7)
- added C37: 100nF, KiCad/Capacitor_SMD.pretty:C_0402_1005Metric_Pad0.74x0.62mm_HandSolder, F.Cu at (49.3, 15.7)
- added J1: PicoBlade, KiCad/Connector_Molex.pretty:Molex_PicoBlade_53261-0571_1x05-1MP_P1.25mm_Horizontal, F.Cu at (20.8, 10.5)
- added J2: PicoBlade, KiCad/Connector_Molex.pretty:Molex_PicoBlade_53261-0571_1x05-1MP_P1.25mm_Horizontal, F.Cu at (20.8, 18.3)
- added J3: USB_C_Receptacle, KiCad/Connector_USB.pretty:USB_C_Receptacle_GCT_USB4105-xx-A_16P_TopMnt_Horizontal, F.Cu at (19.5, 31.9)
- added JP1: TERM, KiCad/Jumper.pretty:SolderJumper-2_P1.3mm_Open_RoundedPad1.0x1.5mm, F.Cu at (30.1, 8.02)
- added Q1: BSS123, KiCad/Package_TO_SOT_SMD.pretty:SOT-23, F.Cu at (50.1, 8.47)
- added R10: 10k, KiCad/Resistor_SMD.pretty:R_0402_1005Metric, F.Cu at (64.3, 29.4)
- added R11: 44.2k, KiCad/Resistor_SMD.pretty:R_0402_1005Metric, F.Cu at (61.4, 28.6)
- added R12: 232k, KiCad/Resistor_SMD.pretty:R_0402_1005Metric, F.Cu at (73.5, 21.0)
- added R13: 10k, KiCad/Resistor_SMD.pretty:R_0402_1005Metric, F.Cu at (70.6, 21.0)
- added R14: 1k, KiCad/Resistor_SMD.pretty:R_0402_1005Metric, F.Cu at (55.5, 15.7)
- added R15: 22k, KiCad/Resistor_SMD.pretty:R_0402_1005Metric, F.Cu at (57.7, 11.3)
- added R16: 1k, KiCad/Resistor_SMD.pretty:R_0402_1005Metric, F.Cu at (62.1, 9.23)
- added R17: 91k, KiCad/Resistor_SMD.pretty:R_0402_1005Metric, F.Cu at (57.7, 13.3)
- added R18: 10k, KiCad/Resistor_SMD.pretty:R_0402_1005Metric, F.Cu at (60.6, 11.3)
- added R19: 91k, KiCad/Resistor_SMD.pretty:R_0402_1005Metric, F.Cu at (65.0, 7.24)
- added R20: 10k, KiCad/Resistor_SMD.pretty:R_0402_1005Metric, F.Cu at (62.1, 7.24)
- added TP1: TestPoint, tunaf1sh/misc.pretty:TestPoint_Pad_D1.0mm_Tight, F.Cu at (33.4, 7.41)
- added TP10: TestPoint, tunaf1sh/misc.pretty:TestPoint_Pad_D1.0mm_Tight, F.Cu at (26.5, 35.1)
- added TP11: TestPoint, tunaf1sh/misc.pretty:TestPoint_Pad_D1.0mm_Tight, F.Cu at (31.3, 27.8)
- added TP12: TestPoint, tunaf1sh/misc.pretty:TestPoint_Pad_D1.0mm_Tight, F.Cu at (17.2, 37.8)
- added TP13: TestPoint, tunaf1sh/misc.pretty:TestPoint_Pad_D1.0mm_Tight, F.Cu at (69.8, 25.1)
- added TP14: TestPoint, KiCad/TestPoint.pretty:TestPoint_Pad_D2.0mm, F.Cu at (58.6, 8.27)
- added TP15: TestPoint, KiCad/TestPoint.pretty:TestPoint_Pad_D2.0mm, F.Cu at (54.2, 12.7)
- added TP16: TestPoint, KiCad/TestPoint.pretty:TestPoint_Pad_D2.0mm, F.Cu at (54.6, 8.27)
- added TP2: TestPoint, tunaf1sh/misc.pretty:TestPoint_Pad_D1.0mm_Tight, F.Cu at (29.1, 13.3)
- added TP3: TestPoint, tunaf1sh/misc.pretty:TestPoint_Pad_D1.0mm_Tight, F.Cu at (31.4, 11.0)
- added TP4: TestPoint, tunaf1sh/misc.pretty:TestPoint_Pad_D1.0mm_Tight, F.Cu at (29.1, 11.0)
- added TP5: TestPoint, tunaf1sh/misc.pretty:TestPoint_Pad_D1.0mm_Tight, F.Cu at (48.3, 34.8)
- added TP6: TestPoint, tunaf1sh/misc.pretty:TestPoint_Pad_D1.0mm_Tight, F.Cu at (52.3, 32.3)
- added TP7: TestPoint, tunaf1sh/misc.pretty:TestPoint_Pad_D1.0mm_Tight, F.Cu at (19.5, 37.8)
- added TP8: TestPoint, tunaf1sh/misc.pretty:TestPoint_Pad_D1.0mm_Tight, F.Cu at (26.5, 37.4)
- added TP9: TestPoint, tunaf1sh/misc.pretty:TestPoint_Pad_D1.0mm_Tight, F.Cu at (14.8, 37.8)
- added U3: MCP25625-E/ML, tunaf1sh/QFN.pretty:QFN-28L, F.Cu at (43.3, 30.5)
- added U5: 74CBTLV3245BQ, tunaf1sh/snapeda.pretty:QFN50P450X250X100-21N, F.Cu at (27.8, 30.6)
- added U6: LMZ21700SILR, tunaf1sh/snapeda.pretty:CONV_TPS82140SILR, F.Cu at (62.6, 22.3)
- added U7: SiP32432DR3, KiCad/Package_TO_SOT_SMD.pretty:SOT-363_SC-70-6, F.Cu at (66.6, 26.5)
- added U8: LSM6DSL, KiCad/Package_LGA.pretty:LGA-14_3x2.5mm_P0.5mm_LayoutBorder3x4y, F.Cu at (49.9, 12.7)
- added Y1: 16MHz, KiCad/Crystal.pretty:Crystal_SMD_3225-4Pin_3.2x2.5mm, F.Cu at (49.7, 28.9)
- C31: value 10nF -> 100nF
- C33: value 100nF -> 10nF
- D2: value LED -> AAA3528; footprint LED_SMD:LED_0603_1608Metric -> KiCad/LED_SMD.pretty:LED_Kingbright_AAA3528ESGCT
- D3: value LED -> DESD2CAN; footprint LED_SMD:LED_0603_1608Metric -> KiCad/Package_TO_SOT_SMD.pretty:SOT-23
- D4: value LED -> MBR0540; footprint LED_SMD:LED_0603_1608Metric -> KiCad/Diode_SMD.pretty:D_SOD-123
- D5: value LED -> SD24-7; footprint LED_SMD:LED_0603_1608Metric -> KiCad/Diode_SMD.pretty:D_SOD-323
- R2, R3: value 10K -> 1k; footprint MCU_Nordic_Accessory:R_0201 -> KiCad/Resistor_SMD.pretty:R_0402_1005Metric
- R4: value 0 -> 1k; footprint MCU_Nordic_Accessory:R_0201 -> KiCad/Resistor_SMD.pretty:R_0402_1005Metric
- R5: value 0 -> 120R; footprint MCU_Nordic_Accessory:R_0201 -> KiCad/Resistor_SMD.pretty:R_0603_1608Metric
- R6: value 220 -> 1k; footprint MCU_Nordic_Accessory:R_0402 -> KiCad/Resistor_SMD.pretty:R_0603_1608Metric
- R7, R8: value 220 -> 5k1; footprint MCU_Nordic_Accessory:R_0402 -> KiCad/Resistor_SMD.pretty:R_0402_1005Metric
- R9: value 220 -> 50k; footprint MCU_Nordic_Accessory:R_0402 -> KiCad/Resistor_SMD.pretty:R_0402_1005Metric
- U2: footprint MCU_Nordic_Accessory:SOP-8_3.9x4.9mm_P1.27mm -> KiCad/Package_SON.pretty:WSON-8-1EP_6x5mm_P1.27mm_EP3.4x4mm
- U4: value SHTC3 -> SN74LVC1G00DRY2; footprint MCU_Nordic_Accessory:Sensirion_DFN-4-1EP_2x2mm_P1mm_EP0.7x1.6mm -> digikey/digikey-kicad-library/digikey-footprints.pretty:UFDFN-6_1.45x1mm
Connections:
- net /SHIELD renamed /USB/SHIELD
- net /VBUS_CONN renamed /USB/VBUS_CONN
- C10 pad 1: VDD -> VCC
- C11 pad 1: VDD -> VCC
- C12 pad 1: VDD -> VCC
- C13 pad 1: VDD -> VCC
- C14 pad 1: VDD -> VCC
- C15 pad 1: VDD -> VCC
- C16 pad 1: VDD -> VCC
- C19 pad 1: VDD -> VCC
- C20 pad 1: VDD -> VCC
- C21 pad 1: VDD -> VCC
- C22 pad 1: /VDDH -> /Radio Sheet/VDDH
- C8 pad 1: VDD -> VCC
- C9 pad 1: VDD -> VCC
- D1 pad 2: /D*_N -> /Radio Sheet/D_P
- D1 pad 3: /D*_P -> /Radio Sheet/D_N
- D2 pad 1: /P1.11 -> Net-(D2-Pad1)
- D2 pad 2: Net-(D2-Pad2) -> VCC
- D3 pad 1: /P1.12 -> /CAN_L
- D3 pad 2: Net-(D3-Pad2) -> /CAN_H
- D4 pad 1: /P1.13 -> Net-(C28-Pad1)
- D4 pad 2: Net-(D4-Pad2) -> +12V
- D5 pad 1: /P1.14 -> Net-(D5-Pad1)
- D5 pad 2: Net-(D5-Pad2) -> GND
- FB2 pad 1: /USB_GND -> /USB/USB_GND
- L4 pad 2: VDD -> VCC
- R2 pad 1: VDD -> Net-(D2-Pad1)
- R2 pad 2: /P1.02/I2C -> /P1.00
- R3 pad 1: VDD -> Net-(D2-Pad3)
- R3 pad 2: /P1.03/I2C -> /P1.01
- R4 pad 1: /VDDH_EXT -> Net-(D2-Pad4)
- R4 pad 2: /VDDH -> /P1.04
- R5 pad 1: /VDD_EXT -> Net-(JP1-Pad2)
- R5 pad 2: VDD -> /CAN_L
- R6 pad 1: Net-(D2-Pad2) -> VDD
- R6 pad 2: VDD -> /P0.30
- R7 pad 1: Net-(D3-Pad2) -> /USB/CC1
- R7 pad 2: VDD -> GND
- R8 pad 1: Net-(D4-Pad2) -> /USB/CC2
- R8 pad 2: VDD -> GND
- R9 pad 1: Net-(D5-Pad2) -> +12V
- R9 pad 2: VDD -> /P0.26/AIN5
- SWD1 pad 1: VDD -> VCC
- U1 pad A19: VDD -> VCC
- U1 pad AC1: VDD -> VCC
- U1 pad AG1: VDD -> VCC
- U1 pad AJ31: VDD -> VCC
- U1 pad AL11: VDD -> VCC
- U1 pad AL17: VDD -> VCC
- U1 pad AL25: VDD -> VCC
- U1 pad AL3: VDD -> VCC
- U1 pad AL7: VDD -> VCC
- U1 pad B28: VDD -> VCC
- U1 pad B8: VDD -> VCC
- U1 pad C1: VDD -> VCC
- U1 pad E1: /VDDH -> /Radio Sheet/VDDH
- U1 pad E31: VDD -> VCC
- U1 pad L1: VDD -> VCC
- U1 pad N31: VDD -> VCC
- U1 pad U1: VDD -> VCC
- U2 pad 8: VDD -> VCC
- U4 pad 1: VDD -> /USB/CC1
- U4 pad 2: /P1.02/I2C -> /USB/CC2
- U4 pad 3: /P1.03/I2C -> GND
- U4 pad 4: GND -> /USB/DBG_EN
- U4 pad 5: GND -> VCC
Routing:
- net VDD: track 141.9 -> 1.44 mm, vias 17 -> 0
- net VCC: track 0.00 -> 112.8 mm, vias 0 -> 17
- net /Radio Sheet/D_P: track 10.9 -> 63.1 mm
- net /D*_N: track 52.2 -> 0.00 mm
- net /D*_P: track 52.0 -> 0.00 mm
- net /Radio Sheet/D_N: track 11.0 -> 63.0 mm
- net Net-(JP1-Pad2): track 0.00 -> 47.8 mm, vias 0 -> 2
- net /VDD_EXT: track 47.8 -> 0.00 mm, vias 2 -> 0
- net Net-(D2-Pad4): track 0.00 -> 32.2 mm, vias 0 -> 2
- net /VDDH_EXT: track 32.2 -> 0.00 mm, vias 2 -> 0
- net /CAN_L: track 0.00 -> 11.4 mm
- net /P1.02/I2C: track 57.5 -> 46.8 mm
- net /P1.00: track 45.1 -> 55.8 mm
- net /P1.03/I2C: track 56.2 -> 46.7 mm
- net /P1.01: track 47.3 -> 56.7 mm
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