File: spirit_logger_hardware.kicad_pcb (KiCad board)
At the start: 4 copper layers, 25 x 61.5 mm, 117 parts, among them J1 PicoBlade, J2 PicoBlade, J3 USB_C_Receptacle, Q1 BSS123, U1 nRF5340-QKAA, U2 MX25R6435F, U3 MCP25625-E/ML, U4 SN74LVC1G00DRY2, U5 74CBTLV3245BQ, U6 LMZ21700SILR, U7 SiP32432DR3, U8 LSM6DSL, X1 Crystal_GND24, X2 Crystal, Y1 16MHz

Commit message: update BoM
Parts:
- added G***: LOGO, tuna-f1sh/jbr-kicad/Logos.pretty:specialized_xs, F.Cu at (92.8, 52.0)
- C1, C10, C11, C12, C13, C14, C15, C19, C23, C24, C25, C26, C27, C29, C30, C31, C32, C33, C36, C37, C4, C6, C8, C9: footprint MCU_Nordic_Accessory:C_0201 -> Capacitor_SMD:C_0201_0603Metric
- C16, C20, C3, C5, C7: footprint MCU_Nordic_Accessory:C_0402 -> Capacitor_SMD:C_0402_1005Metric
- C17, C18, C21, C22, C34: footprint MCU_Nordic_Accessory:C_0603 -> Capacitor_SMD:C_0603_1608Metric
- C2: value N/C -> 0uF; footprint MCU_Nordic_Accessory:C_0201 -> Capacitor_SMD:C_0201_0603Metric
- D1: footprint MCU_Nordic_Accessory:SOT-143 -> Package_TO_SOT_SMD:SOT-143
- FB1, FB2, FB3: footprint MCU_Nordic_Accessory:FB_0603 -> Inductor_SMD:L_0603_1608Metric
- L1: footprint MCU_Nordic_Accessory:L_0201 -> Inductor_SMD:L_0201_0603Metric
- L2, L3, L4: footprint MCU_Nordic_Accessory:L_0603 -> Inductor_SMD:L_0603_1608Metric
- R1: footprint MCU_Nordic_Accessory:R_0201 -> Resistor_SMD:R_0201_0603Metric
- X1: footprint MCU_Nordic_Accessory:XTAL_32M_4PIN -> Crystal:Crystal_SMD_2016-4Pin_2.0x1.6mm
- X2: value Crystal -> 32kHz; footprint MCU_Nordic_Accessory:XTAL_32768Hz_2PIN -> Crystal:Crystal_SMD_MicroCrystal_CM9V-T1A-2Pin_1.6x1.0mm
- moved TP11 6.77 mm to (91.5, 78.6)
- moved C27 2.17 mm to (96.4, 89.7), turned to -90 degrees
- moved R1 1.40 mm to (92.3, 67.9), turned to 90 degrees
- moved C20 0.72 mm to (96.2, 67.2)
- moved C32 0.55 mm to (92.3, 86.0)
- moved L2 0.50 mm to (102.4, 67.1)
- moved C2 0.46 mm to (105.5, 72.1)
- moved C30 0.38 mm to (93.0, 93.5)
- moved L3 0.36 mm to (98.3, 66.5)
- moved C8 0.35 mm to (94.5, 70.0), turned to 180 degrees
- moved L4 0.34 mm to (91.7, 73.4)
- moved FB1 0.34 mm to (93.0, 84.9)
- moved C17 0.33 mm to (93.4, 67.6)
- moved C31 0.31 mm to (93.5, 86.3)
- moved C21 0.28 mm to (93.2, 73.6)
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Connections:
- X2 pad 1: /Radio Sheet/XL2 -> /Radio Sheet/XL1
- X2 pad 2: /Radio Sheet/XL1 -> /Radio Sheet/XL2
Routing:
- net VCC: track 135.8 -> 139.7 mm
- net /USB/VBUS_CONN: track 49.4 -> 51.8 mm
- net VBUS: track 39.2 -> 37.4 mm
- net GND: track 43.0 -> 41.6 mm, vias 83 -> 82
- net +5V: track 26.4 -> 25.1 mm
- net /Radio Sheet/VBUS_NET: track 5.07 -> 5.93 mm
- net /Radio Sheet/DECD: track 3.50 -> 4.12 mm
Other:
- board text added: "J.Whittington - Specialized Europe GmbH"
- board text added: "Spirit Logger R${REVISION}"

Commit message: pre-production checks
Parts:
- added G***: LOGO, tuna-f1sh/jbr-kicad/Logos.pretty:specialized_md, B.Cu at (101.7, 70.8)
- moved C9 0.06 mm to (92.6, 77.4)
