File: spirit_logger_hardware.kicad_sch (KiCad schematic)
At the start: 17 parts, among them U2 MX25R6435F

Commit message: rename; annotate and import to pcb
Parts:
- R5: renamed from R?; footprint KiCad/Resistor_SMD.pretty:R_0603_1608Metric_Pad1.05x0.95mm_HandSolder -> KiCad/Resistor_SMD.pretty:R_0603_1608Metric
- gave numbers to parts that had none: 12
Other:
- moved on the sheet: ANT1, D2, R2, R3, R4, SWD1
