File: spirit_logger_hardware.kicad_sch (KiCad schematic)
At the start: 27 parts, among them J1 PicoBlade, J2 PicoBlade, U2 MX25R6435F

Commit message: steps added, before shorten
Parts:
- removed TP22, TP23: TestPoint, tuna-f1sh/jbr-kicad/Misc.pretty:TestPoint_Pad_D1.0mm_Tight, symbol Connector:TestPoint_Small
- J1, J2: symbol Connector:Conn_01x05_Male -> Connector:Conn_01x05_Pin
Connections:
- net CAN_H renamed CAN_P
- net CAN_L renamed CAN_N

Commit message: shortened board with usb-c
Parts:
- added H1, H2, H3, H4: MountingHole, MountingHole:MountingHole_2.2mm_M2_DIN965, symbol Mechanical:MountingHole
Changed lines of the file:
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@@
+    )
+  )
+  (symbol (lib_id "Mechanical:MountingHole") (at 248.8692 264.3124 0) (unit 1)
+    (in_bom yes) (on_board yes) (dnp no) (fields_autoplaced)
+    (property "Reference" "H1" (at 251.4092 263.6687 0)
+      (effects (font (size 1.27 1.27)) (justify left) hide)
+    )
+    (property "Value" "MountingHole" (at 251.4092 265.5897 0)
+      (effects (font (size 1.27 1.27)) (justify left) hide)
+    )
+    (property "Footprint" "MountingHole:MountingHole_2.2mm_M2_DIN965" (at 248.8692 264.3124 0)
+      (effects (font (size 1.27 1.27)) hide)
+    )
+    (property "Datasheet" "~" (at 248.8692 264.3124 0)
+      (effects (font (size 1.27 1.27)) hide)
+    )
+    (property "MFN" "" (at 248.8692 264.3124 0)
+      (effects (font (size 1.27 1.27)) hide)
+    )
+    (property "MPN" "" (at 248.8692 264.3124 0)
+      (effects (font (size 1.27 1.27)) hide)
+    )
+    (property "Description" "" (at 248.8692 264.3124 0)
+      (effects (font (size 1.27 1.27)) hide)
+    )
+    (property "Notes" "" (at 248.8692 264.3124 0)
+      (effects (font (size 1.27 1.27)) hide)
+    )
+    (property "Config" "nofit" (at 248.8692 264.3124 0)
+      (effects (font (size 1.27 1.27)) hide)
+    )
+    (property "Vendor" "" (at 248.8692 264.3124 0)
+      (effects (font (size 1.27 1.27)) hide)
+    )
+    (property "SKU" "" (at 248.8692 264.3124 0)
+      (effects (font (size 1.27 1.27)) hide)
+    )
+    (property "Characteristics" "" (at 248.8692 264.3124 0)
+      (effects (font (size 1.27 1.27)) hide)
+    )
+    (instances
+      (project "spirit_logger_hardware"
+        (path "/e63e39d7-6ac0-4ffd-8aa3-1841a4541b55"
+          (reference "H1") (unit 1)
+        )
+      )
     )
   )
@@
     )
   )
+  (symbol (lib_id "Mechanical:MountingHole") (at 255.6256 264.3124 0) (unit 1)
+    (in_bom yes) (on_board yes) (dnp no) (fields_autoplaced)
+    (property "Reference" "H2" (at 258.1656 263.6687 0)
+      (effects (font (size 1.27 1.27)) (justify left) hide)
+    )
+    (property "Value" "MountingHole" (at 258.1656 265.5897 0)
+      (effects (font (size 1.27 1.27)) (justify left) hide)
+    )
+    (property "Footprint" "MountingHole:MountingHole_2.2mm_M2_DIN965" (at 255.6256 264.3124 0)
+      (effects (font (size 1.27 1.27)) hide)
+    )
+    (property "Datasheet" "~" (at 255.6256 264.3124 0)
+      (effects (font (size 1.27 1.27)) hide)
+    )
+    (property "MFN" "" (at 255.6256 264.3124 0)
+      (effects (font (size 1.27 1.27)) hide)
+    )
+    (property "MPN" "" (at 255.6256 264.3124 0)
+      (effects (font (size 1.27 1.27)) hide)
+    )
+    (property "Description" "" (at 255.6256 264.3124 0)
+      (effects (font (size 1.27 1.27)) hide)
+    )
+    (property "Notes" "" (at 255.6256 264.3124 0)
+      (effects (font (size 1.27 1.27)) hide)
+    )
+    (property "Config" "nofit" (at 255.6256 264.3124 0)
+      (effects (font (size 1.27 1.27)) hide)
+    )
+    (property "Vendor" "" (at 255.6256 264.3124 0)
+      (effects (font (size 1.27 1.27)) hide)
+    )
+    (property "SKU" "" (at 255.6256 264.3124 0)
+      (effects (font (size 1.27 1.27)) hide)
+    )
+    (property "Characteristics" "" (at 255.6256 264.3124 0)
+      (effects (font (size 1.27 1.27)) hide)
+    )
+    (instances
+      (project "spirit_logger_hardware"
+        (path "/e63e39d7-6ac0-4ffd-8aa3-1841a4541b55"
+          (reference "H2") (unit 1)
+        )
+      )
+    )
+  )
   (symbol (lib_id "Device:R_Small") (at 371.602 148.4884 0) (unit 1)
     (in_bom yes) (on_board yes) (dnp no)
@@
     )
   )
+  (symbol (lib_id "Mechanical:MountingHole") (at 255.6764 270.51 0) (unit 1)
+    (in_bom yes) (on_board yes) (dnp no) (fields_autoplaced)
+    (property "Reference" "H4" (at 258.2164 269.8663 0)
+      (effects (font (size 1.27 1.27)) (justify left) hide)
+    )
+    (property "Value" "MountingHole" (at 258.2164 271.7873 0)
+      (effects (font (size 1.27 1.27)) (justify left) hide)
+    )
+    (property "Footprint" "MountingHole:MountingHole_2.2mm_M2_DIN965" (at 255.6764 270.51 0)
+      (effects (font (size 1.27 1.27)) hide)
+    )
+    (property "Datasheet" "~" (at 255.6764 270.51 0)
+      (effects (font (size 1.27 1.27)) hide)
+    )
+    (property "MFN" "" (at 255.6764 270.51 0)
+      (effects (font (size 1.27 1.27)) hide)
+    )
+    (property "MPN" "" (at 255.6764 270.51 0)
+      (effects (font (size 1.27 1.27)) hide)
+    )
+    (property "Description" "" (at 255.6764 270.51 0)
+      (effects (font (size 1.27 1.27)) hide)
+    )
+    (property "Notes" "" (at 255.6764 270.51 0)
+      (effects (font (size 1.27 1.27)) hide)
+    )
+    (property "Config" "nofit" (at 255.6764 270.51 0)
+      (effects (font (size 1.27 1.27)) hide)
+    )
+    (property "Vendor" "" (at 255.6764 270.51 0)
+      (effects (font (size 1.27 1.27)) hide)
+    )
+    (property "SKU" "" (at 255.6764 270.51 0)
+      (effects (font (size 1.27 1.27)) hide)
+    )
+    (property "Characteristics" "" (at 255.6764 270.51 0)
+      (effects (font (size 1.27 1.27)) hide)
+    )
+    (instances
+      (project "spirit_logger_hardware"
+        (path "/e63e39d7-6ac0-4ffd-8aa3-1841a4541b55"
+          (reference "H4") (unit 1)
+        )
+      )
+    )
+  )
   (symbol (lib_id "Connector:TestPoint_Small") (at 185.4708 238.1504 0) (unit 1)
     (in_bom yes) (on_board yes) (dnp no)
@@
         )
       )
+    )
+  )
+  (symbol (lib_id "Mechanical:MountingHole") (at 248.8692 270.51 0) (unit 1)
+    (in_bom yes) (on_board yes) (dnp no) (fields_autoplaced)
+    (property "Reference" "H3" (at 251.4092 269.8663 0)
+      (effects (font (size 1.27 1.27)) (justify left) hide)
+    )
+    (property "Value" "MountingHole" (at 251.4092 271.7873 0)
+      (effects (font (size 1.27 1.27)) (justify left) hide)
+    )
+    (property "Footprint" "MountingHole:MountingHole_2.2mm_M2_DIN965" (at 248.8692 270.51 0)
+      (effects (font (size 1.27 1.27)) hide)
+    )
+    (property "Datasheet" "~" (at 248.8692 270.51 0)
+      (effects (font (size 1.27 1.27)) hide)
+    )
+    (property "MFN" "" (at 248.8692 270.51 0)
+      (effects (font (size 1.27 1.27)) hide)
+    )
+    (property "MPN" "" (at 248.8692 270.51 0)
+      (effects (font (size 1.27 1.27)) hide)
+    )
+    (property "Description" "" (at 248.8692 270.51 0)
+      (effects (font (size 1.27 1.27)) hide)
+    )
+    (property "Notes" "" (at 248.8692 270.51 0)
+      (effects (font (size 1.27 1.27)) hide)
+    )
+    (property "Config" "nofit" (at 248.8692 270.51 0)
+      (effects (font (size 1.27 1.27)) hide)
+    )
+    (property "Vendor" "" (at 248.8692 270.51 0)
+      (effects (font (size 1.27 1.27)) hide)
+    )
+    (property "SKU" "" (at 248.8692 270.51 0)
+      (effects (font (size 1.27 1.27)) hide)
+    )
+    (property "Characteristics" "" (at 248.8692 270.51 0)
+      (effects (font (size 1.27 1.27)) hide)
+    )
+    (instances
+      (project "spirit_logger_hardware"
+        (path "/e63e39d7-6ac0-4ffd-8aa3-1841a4541b55"
+          (reference "H3") (unit 1)
+        )
+      )

Commit message: before removal of Nordic passive footprints
Parts:
- C19: footprint MCU_Nordic_Accessory:C_0201 -> Capacitor_SMD:C_0201_0603Metric
Changed lines of the file:
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@@
       (effects (font (size 1.27 1.27)) (justify left))
     )
-    (property "Footprint" "MCU_Nordic_Accessory:C_0201" (at 378.0536 218.948 0)
+    (property "Footprint" "Capacitor_SMD:C_0201_0603Metric" (at 378.0536 218.948 0)
       (effects (font (size 1.27 1.27)) hide)
     )

Commit message: update BoM
Parts:
- ANT1: Config (none) -> nofit; now left out of the parts list
- C19: Characteristics (none) -> X7R 6V
- H1, H2, H3, H4: now left out of the parts list
- JP1: MFN (none) -> Amphenol ICC (Commercial Products); MPN (none) -> 12401832E402A; SKU (none) -> 12401832E402ACT-ND; Vendor (none) -> Digikey
- SWD1: Config (none) -> nofit
Changed lines of the file:
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@@
   )
   (symbol (lib_id "Mechanical:MountingHole") (at 248.8692 264.3124 0) (unit 1)
-    (in_bom yes) (on_board yes) (dnp no) (fields_autoplaced)
+    (in_bom no) (on_board yes) (dnp no) (fields_autoplaced)
     (property "Reference" "H1" (at 251.4092 263.6687 0)
       (effects (font (size 1.27 1.27)) (justify left) hide)
@@
       (effects (font (size 1.27 1.27)) hide)
     )
+    (property "Characteristics" "X7R 6V" (at 377.0884 215.138 0)
+      (effects (font (size 1.27 1.27)) hide)
+    )
     (pin "1")
     (pin "2")
@@
       (effects (font (size 1.27 1.27)) hide)
     )
+    (property "MFN" "Amphenol ICC (Commercial Products)" (at 371.602 142.1384 0)
+      (effects (font (size 1.27 1.27)) hide)
+    )
+    (property "MPN" "12401832E402A" (at 371.602 142.1384 0)
+      (effects (font (size 1.27 1.27)) hide)
+    )
+    (property "SKU" "12401832E402ACT-ND" (at 371.602 142.1384 0)
+      (effects (font (size 1.27 1.27)) hide)
+    )
+    (property "Vendor" "Digikey" (at 371.602 142.1384 0)
+      (effects (font (size 1.27 1.27)) hide)
+    )
     (pin "1")
     (pin "2")
@@
     )
     (property "SKU" "1092-1201-ND" (at 355.4984 213.868 0)
+      (effects (font (size 1.27 1.27)) hide)
+    )
+    (property "Description" "FLASH - NOR Memory IC 64Mbit SPI - Quad I/O 80 MHz 8-WSON (6x5)" (at 355.4984 213.868 0)
       (effects (font (size 1.27 1.27)) hide)
     )
@@
       (effects (font (size 1.27 1.27)) hide)
     )
+    (property "Config" "nofit" (at 130.8608 59.7916 0)
+      (effects (font (size 1.27 1.27)) hide)
+    )
     (pin "1")
     (pin "2")
@@
   )
   (symbol (lib_id "MCU_Nordic_Custom:Antenna_L") (at 237.617 47.0916 0) (unit 1)
-    (in_bom yes) (on_board yes) (dnp no) (fields_autoplaced)
+    (in_bom no) (on_board yes) (dnp no) (fields_autoplaced)
     (property "Reference" "ANT1" (at 241.427 43.2815 0)
       (effects (font (size 1.27 1.27)) (justify left))
@@
     )
     (property "Datasheet" "" (at 237.617 47.0916 0)
+      (effects (font (size 1.27 1.27)) hide)
+    )
+    (property "Config" "nofit" (at 237.617 47.0916 0)
+      (effects (font (size 1.27 1.27)) hide)
+    )
+    (property "MFN" "" (at 237.617 47.0916 0)
+      (effects (font (size 1.27 1.27)) hide)
+    )
+    (property "MPN" "" (at 237.617 47.0916 0)
+      (effects (font (size 1.27 1.27)) hide)
+    )
+    (property "Description" "" (at 237.617 47.0916 0)
+      (effects (font (size 1.27 1.27)) hide)
+    )
+    (property "Notes" "" (at 237.617 47.0916 0)
+      (effects (font (size 1.27 1.27)) hide)
+    )
+    (property "Vendor" "" (at 237.617 47.0916 0)
+      (effects (font (size 1.27 1.27)) hide)
+    )
+    (property "SKU" "" (at 237.617 47.0916 0)
+      (effects (font (size 1.27 1.27)) hide)
+    )
+    (property "Characteristics" "" (at 237.617 47.0916 0)
       (effects (font (size 1.27 1.27)) hide)
     )
@@
   )
   (symbol (lib_id "Mechanical:MountingHole") (at 255.6256 264.3124 0) (unit 1)
-    (in_bom yes) (on_board yes) (dnp no) (fields_autoplaced)
+    (in_bom no) (on_board yes) (dnp no) (fields_autoplaced)
     (property "Reference" "H2" (at 258.1656 263.6687 0)
       (effects (font (size 1.27 1.27)) (justify left) hide)
@@
   )
   (symbol (lib_id "Mechanical:MountingHole") (at 255.6764 270.51 0) (unit 1)
-    (in_bom yes) (on_board yes) (dnp no) (fields_autoplaced)
+    (in_bom no) (on_board yes) (dnp no) (fields_autoplaced)
     (property "Reference" "H4" (at 258.2164 269.8663 0)
       (effects (font (size 1.27 1.27)) (justify left) hide)
@@
   )
   (symbol (lib_id "Mechanical:MountingHole") (at 248.8692 270.51 0) (unit 1)
-    (in_bom yes) (on_board yes) (dnp no) (fields_autoplaced)
+    (in_bom no) (on_board yes) (dnp no) (fields_autoplaced)
     (property "Reference" "H3" (at 251.4092 269.8663 0)
       (effects (font (size 1.27 1.27)) (justify left) hide)

Commit message: production files sent
Parts:
- D3: MFN DESD2CAN2SOQ-7 -> Diodes Incorporated; MPN Diodes Incorporated -> DESD2CAN2SOQ-7
Changed lines of the file:
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@@
       (effects (font (size 1.27 1.27)) hide)
     )
-    (property "MFN" "DESD2CAN2SOQ-7" (at 363.982 162.7124 0)
+    (property "MFN" "Diodes Incorporated" (at 363.982 162.7124 0)
       (effects (font (size 1.27 1.27)) hide)
     )
-    (property "MPN" "Diodes Incorporated" (at 363.982 162.7124 0)
+    (property "MPN" "DESD2CAN2SOQ-7" (at 363.982 162.7124 0)
       (effects (font (size 1.27 1.27)) hide)
     )

Commit message: makefile
Parts:
- JP1: MFN Amphenol ICC (Commercial Products) -> (none); MPN 12401832E402A -> (none); SKU 12401832E402ACT-ND -> (none); Vendor Digikey -> (none)
Changed lines of the file:
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@@
       (effects (font (size 1.27 1.27)) hide)
     )
-    (property "MFN" "Amphenol ICC (Commercial Products)" (at 371.602 142.1384 0)
+    (property "MFN" "" (at 371.602 142.1384 0)
       (effects (font (size 1.27 1.27)) hide)
     )
-    (property "MPN" "12401832E402A" (at 371.602 142.1384 0)
+    (property "MPN" "" (at 371.602 142.1384 0)
       (effects (font (size 1.27 1.27)) hide)
     )
-    (property "SKU" "12401832E402ACT-ND" (at 371.602 142.1384 0)
+    (property "SKU" "" (at 371.602 142.1384 0)
       (effects (font (size 1.27 1.27)) hide)
     )
-    (property "Vendor" "Digikey" (at 371.602 142.1384 0)
+    (property "Vendor" "" (at 371.602 142.1384 0)
       (effects (font (size 1.27 1.27)) hide)
     )
