File: Radio.kicad_sch (KiCad schematic)
At the start: 29 parts, among them U1 nRF5340-QKAA, X1 Crystal_GND24, X2 Crystal

Commit message: drc updated for pcbway advanced; layout and tidy
Changed lines of the file:
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@@
   (junction (at 208.788 92.1004) (diameter 0) (color 0 0 0 0)
   )
-  (junction (at 132.588 111.1504) (diameter 0) (color 0 0 0 0)
-  )
   (junction (at 208.788 107.3404) (diameter 0) (color 0 0 0 0)
   )
@@
     (stroke (width 0) (type default) (color 0 0 0 0))
   )
-  (wire (pts (xy 132.588 107.3404) (xy 132.588 111.1504))
-    (stroke (width 0) (type default) (color 0 0 0 0))
-  )
   (wire (pts (xy 93.218 92.1004) (xy 93.218 81.9404))
     (stroke (width 0) (type default) (color 0 0 0 0))
@@
     (stroke (width 0) (type default) (color 0 0 0 0))
   )
-  (wire (pts (xy 94.488 111.1504) (xy 132.588 111.1504))
+  (wire (pts (xy 94.488 111.1504) (xy 140.208 111.1504))
     (stroke (width 0) (type default) (color 0 0 0 0))
   )
@@
   )
   (wire (pts (xy 281.178 187.3504) (xy 291.338 187.3504))
-    (stroke (width 0) (type default) (color 0 0 0 0))
-  )
-  (wire (pts (xy 132.588 111.1504) (xy 140.208 111.1504))
     (stroke (width 0) (type default) (color 0 0 0 0))
   )
@@
       (effects (font (size 1.27 1.27)) hide)
     )
-    (pin "1")
-  )
-  (symbol (lib_id "power:VDD") (at 132.588 107.3404 0) (unit 1)
-    (in_bom yes) (on_board yes) (fields_autoplaced)
-    (property "Reference" "#PWR06" (id 0) (at 132.588 111.1504 0)
-      (effects (font (size 1.27 1.27)) hide)
-    )
-    (property "Value" "VDD" (id 1) (at 132.588 102.2604 0))
-    (property "Footprint" "" (id 2) (at 132.588 107.3404 0)
-      (effects (font (size 1.27 1.27)) hide)
-    )
-    (property "Datasheet" "" (id 3) (at 132.588 107.3404 0)
-      (effects (font (size 1.27 1.27)) hide)
-    )

Commit message: steps added, before shorten
Parts:
- U1: footprint footprints_nordic:Nordic-AQFN-1EP_7x7mm_P0.4mm -> MCU_Nordic_Custom:Nordic-AQFN-1EP_7x7mm_P0.4mm
Connections:
- net VDD: now also C10.1, C11.1, C12.1, C13.1, C14.1, C15.1, C8.1, C9.1, U1.AC1 (VDD), U1.AG1 (VDD), U1.AJ31 (VDD), U1.AL11 (VDD), U1.AL17 (VDD), U1.AL25 (VDD), U1.AL3 (VDD), U1.AL7 (VDD), U1.B28 (VDD), U1.C1 (VDD), U1.E31 (VDD), U1.N31 (VDD), U1.U1 (VDD)

Commit message: before removal of Nordic passive footprints
Parts:
- C1, C10, C11, C12, C13, C14, C15, C2, C4, C6, C8, C9: footprint MCU_Nordic_Accessory:C_0201 -> Capacitor_SMD:C_0201_0603Metric
- C16, C20, C3, C5, C7: footprint MCU_Nordic_Accessory:C_0402 -> Capacitor_SMD:C_0402_1005Metric
- C17, C18, C21, C22: footprint MCU_Nordic_Accessory:C_0603 -> Capacitor_SMD:C_0603_1608Metric
- L1: footprint MCU_Nordic_Accessory:L_0201 -> Inductor_SMD:L_0201_0603Metric
- L2, L3, L4: footprint MCU_Nordic_Accessory:L_0603 -> Inductor_SMD:L_0603_1608Metric
- R1: footprint MCU_Nordic_Accessory:R_0201 -> Resistor_SMD:R_0201_0603Metric
Changed lines of the file:
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@@
       (effects (font (size 1.27 1.27)))
     )
-    (property "Footprint" "MCU_Nordic_Accessory:L_0603" (at 114.808 84.4804 0)
+    (property "Footprint" "Inductor_SMD:L_0603_1608Metric" (at 114.808 84.4804 0)
       (effects (font (size 1.27 1.27)) hide)
     )
@@
       (effects (font (size 1.27 1.27)) (justify left))
     )
-    (property "Footprint" "MCU_Nordic_Accessory:C_0201" (at 247.8532 134.0104 0)
+    (property "Footprint" "Capacitor_SMD:C_0201_0603Metric" (at 247.8532 134.0104 0)
       (effects (font (size 1.27 1.27)) hide)
     )
@@
       (effects (font (size 1.27 1.27)) (justify left))
     )
-    (property "Footprint" "MCU_Nordic_Accessory:C_0201" (at 235.1532 134.0104 0)
+    (property "Footprint" "Capacitor_SMD:C_0201_0603Metric" (at 235.1532 134.0104 0)
       (effects (font (size 1.27 1.27)) hide)
     )
@@
       (effects (font (size 1.27 1.27)))
     )
-    (property "Footprint" "MCU_Nordic_Accessory:L_0603" (at 126.238 113.6904 0)
+    (property "Footprint" "Inductor_SMD:L_0603_1608Metric" (at 126.238 113.6904 0)
       (effects (font (size 1.27 1.27)) hide)
     )
@@
       (effects (font (size 1.27 1.27)))
     )
-    (property "Footprint" "MCU_Nordic_Accessory:C_0603" (at 116.078 154.0256 0)
+    (property "Footprint" "Capacitor_SMD:C_0603_1608Metric" (at 116.078 154.0256 0)
       (effects (font (size 1.27 1.27)) hide)
     )
@@
       (effects (font (size 1.27 1.27)) (justify left))
     )
-    (property "Footprint" "MCU_Nordic_Accessory:C_0201" (at 118.3132 99.7204 0)
+    (property "Footprint" "Capacitor_SMD:C_0201_0603Metric" (at 118.3132 99.7204 0)
       (effects (font (size 1.27 1.27)) hide)
     )
@@
       (effects (font (size 1.27 1.27)))
     )
-    (property "Footprint" "MCU_Nordic_Accessory:L_0603" (at 127.508 146.7104 0)
+    (property "Footprint" "Inductor_SMD:L_0603_1608Metric" (at 127.508 146.7104 0)
       (effects (font (size 1.27 1.27)) hide)
     )
@@
       (effects (font (size 1.27 1.27)) (justify left))
     )
-    (property "Footprint" "MCU_Nordic_Accessory:C_0603" (at 95.4532 151.7904 0)
+    (property "Footprint" "Capacitor_SMD:C_0603_1608Metric" (at 95.4532 151.7904 0)
       (effects (font (size 1.27 1.27)) hide)
     )
@@
       (effects (font (size 1.27 1.27)) (justify left))
     )
-    (property "Footprint" "MCU_Nordic_Accessory:C_0201" (at 247.8532 109.8804 0)
+    (property "Footprint" "Capacitor_SMD:C_0201_0603Metric" (at 247.8532 109.8804 0)
       (effects (font (size 1.27 1.27)) hide)
     )
@@
       (effects (font (size 1.27 1.27)) (justify left))
     )
-    (property "Footprint" "MCU_Nordic_Accessory:C_0201" (at 216.1032 92.1004 0)
+    (property "Footprint" "Capacitor_SMD:C_0201_0603Metric" (at 216.1032 92.1004 0)
       (effects (font (size 1.27 1.27)) hide)
     )
@@
       (effects (font (size 1.27 1.27)) (justify left))
     )
-    (property "Footprint" "MCU_Nordic_Accessory:C_0402" (at 95.4532 121.3104 0)
+    (property "Footprint" "Capacitor_SMD:C_0402_1005Metric" (at 95.4532 121.3104 0)
       (effects (font (size 1.27 1.27)) hide)
     )
@@
       (effects (font (size 1.27 1.27)) (justify left))
     )
-    (property "Footprint" "MCU_Nordic_Accessory:C_0201" (at 226.2632 109.8804 0)
+    (property "Footprint" "Capacitor_SMD:C_0201_0603Metric" (at 226.2632 109.8804 0)
       (effects (font (size 1.27 1.27)) hide)
     )
@@
       (effects (font (size 1.27 1.27)) (justify left))
     )
-    (property "Footprint" "MCU_Nordic_Accessory:C_0402" (at 120.8532 134.0104 0)
+    (property "Footprint" "Capacitor_SMD:C_0402_1005Metric" (at 120.8532 134.0104 0)
       (effects (font (size 1.27 1.27)) hide)
     )
@@
       (effects (font (size 1.27 1.27)) (justify left))
     )
-    (property "Footprint" "MCU_Nordic_Accessory:C_0201" (at 226.2632 92.1004 0)
+    (property "Footprint" "Capacitor_SMD:C_0201_0603Metric" (at 226.2632 92.1004 0)
       (effects (font (size 1.27 1.27)) hide)
     )
@@
       (effects (font (size 1.27 1.27)) (justify left))
     )
-    (property "Footprint" "MCU_Nordic_Accessory:C_0402" (at 124.6632 182.2704 0)
+    (property "Footprint" "Capacitor_SMD:C_0402_1005Metric" (at 124.6632 182.2704 0)
       (effects (font (size 1.27 1.27)) hide)
     )
@@
       (effects (font (size 1.27 1.27)) (justify left))
     )
-    (property "Footprint" "MCU_Nordic_Accessory:C_0201" (at 237.6932 109.8804 0)
+    (property "Footprint" "Capacitor_SMD:C_0201_0603Metric" (at 237.6932 109.8804 0)
       (effects (font (size 1.27 1.27)) hide)
     )
@@
       (effects (font (size 1.27 1.27)) (justify left))
     )
-    (property "Footprint" "MCU_Nordic_Accessory:C_0402" (at 94.1832 99.7204 0)
+    (property "Footprint" "Capacitor_SMD:C_0402_1005Metric" (at 94.1832 99.7204 0)
       (effects (font (size 1.27 1.27)) hide)
     )
@@
       (effects (font (size 1.27 1.27)) (justify left))
     )
-    (property "Footprint" "MCU_Nordic_Accessory:C_0402" (at 105.6132 99.7204 0)
+    (property "Footprint" "Capacitor_SMD:C_0402_1005Metric" (at 105.6132 99.7204 0)
       (effects (font (size 1.27 1.27)) hide)
     )
@@
       (effects (font (size 1.27 1.27)) (justify left))
     )
-    (property "Footprint" "MCU_Nordic_Accessory:C_0603" (at 91.6432 182.2704 0)
+    (property "Footprint" "Capacitor_SMD:C_0603_1608Metric" (at 91.6432 182.2704 0)
       (effects (font (size 1.27 1.27)) hide)
     )
@@
       (effects (font (size 1.27 1.27)) (justify left))
     )
-    (property "Footprint" "MCU_Nordic_Accessory:C_0201" (at 216.1032 109.8804 0)
+    (property "Footprint" "Capacitor_SMD:C_0201_0603Metric" (at 216.1032 109.8804 0)
       (effects (font (size 1.27 1.27)) hide)
     )
@@
       (effects (font (size 1.27 1.27)) (justify left))
     )
-    (property "Footprint" "MCU_Nordic_Accessory:C_0201" (at 247.8532 92.1004 0)
+    (property "Footprint" "Capacitor_SMD:C_0201_0603Metric" (at 247.8532 92.1004 0)
       (effects (font (size 1.27 1.27)) hide)
     )
@@
       (effects (font (size 1.27 1.27)) (justify left))
     )
-    (property "Footprint" "MCU_Nordic_Accessory:C_0201" (at 114.5032 182.2704 0)
+    (property "Footprint" "Capacitor_SMD:C_0201_0603Metric" (at 114.5032 182.2704 0)
       (effects (font (size 1.27 1.27)) hide)
     )
@@
       (effects (font (size 1.27 1.27)) (justify left))
     )
-    (property "Footprint" "MCU_Nordic_Accessory:C_0201" (at 237.6932 92.1004 0)
+    (property "Footprint" "Capacitor_SMD:C_0201_0603Metric" (at 237.6932 92.1004 0)
       (effects (font (size 1.27 1.27)) hide)
     )
@@
       (effects (font (size 1.27 1.27)))
     )
-    (property "Footprint" "MCU_Nordic_Accessory:L_0201" (at 240.538 126.3904 0)
+    (property "Footprint" "Inductor_SMD:L_0201_0603Metric" (at 240.538 126.3904 0)
       (effects (font (size 1.27 1.27)) hide)
     )
@@
       (effects (font (size 1.27 1.27)))
     )
-    (property "Footprint" "MCU_Nordic_Accessory:R_0201" (at 83.058 164.9984 90)
+    (property "Footprint" "Resistor_SMD:R_0201_0603Metric" (at 83.058 164.9984 90)
       (effects (font (size 1.27 1.27)) hide)
     )
@@
       (effects (font (size 1.27 1.27)) (justify left))
     )
-    (property "Footprint" "MCU_Nordic_Accessory:C_0603" (at 103.0732 182.2704 0)
-      (effects (font (size 1.27 1.27)) hide)
-    )
+    (property "Footprint" "Capacitor_SMD:C_0603_1608Metric" (at 103.0732 182.2704 0)
+      (effects (font (size 1.27 1.27)) hide)
+    )

Commit message: update BoM
Parts:
- C1: Characteristics (none) -> NPO 6V
- C10, C11, C12, C13, C14, C15, C16, C20, C3, C5, C6, C7, C8, C9: Characteristics (none) -> X7R 6V
- C17, C18, C21, C22: Characteristics (none) -> X5R 25V
- C2: value N/C -> 0uF; Config (none) -> dnf
- C4: Characteristics (none) -> X5R 10V
- L1: value L -> 2.2nH; Characteristics (none) -> High frequency chip inductor, ±5%; MFN (none) -> TE Connectivity Passive Product; MPN (none) -> 36501E2N2JTDG; SKU (none) -> A103705CT-ND; Vendor (none) -> Digikey
- L2, L3, L4: Characteristics (none) -> 80 mA 20%
- R1: Characteristics (none) -> 1%
- U1: MFN (none) -> Nordic Semiconductor ASA; MPN (none) -> NRF5340-QKAA-R; SKU (none) -> 4823-NRF5340-QKAA-RCT-ND; Vendor (none) -> Digikey
- X1: value Crystal_GND24 -> 32MHz; footprint MCU_Nordic_Accessory:XTAL_32M_4PIN -> Crystal:Crystal_SMD_2016-4Pin_2.0x1.6mm; MFN (none) -> ECS Inc.; MPN (none) -> ECS-320-8-37-CKM-TR3; SKU (none) -> 50-ECS-320-8-37-CKM-TR3CT-ND; Vendor (none) -> Digikey
- X2: value Crystal -> 32kHz; footprint MCU_Nordic_Accessory:XTAL_32768Hz_2PIN -> Crystal:Crystal_SMD_MicroCrystal_CM9V-T1A-2Pin_1.6x1.0mm; MFN (none) -> Micro Crystal AG; MPN (none) -> 2195-CM9V-T1A-32.768KHZ-12.5PF-20PPM-TA-QCCT-ND; SKU (none) -> 535-14513-1-ND; Vendor (none) -> Digikey
Connections:
- net XL1: now also X2.1; no longer X2.2
- net XL2: now also X2.2; no longer X2.1
Other:
- moved on the sheet: X2

Commit message: pre-production checks
Other:
- title: Spirit Logger -> Microcontroller
Changed lines of the file:
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@@
   (paper "A3")
   (title_block
-    (title "Spirit Logger")
-    (date "2023-01-23")
+    (title "Microcontroller")
+    (date "2023-02-28")
     (rev "0")
     (company "Specialized Europe GmbH")
+    (comment 1 "J.Whittington 2023")
   )
   (junction (at 119.888 123.8504) (diameter 0) (color 0 0 0 0)

Commit message: makefile
Parts:
- X1: MFN ECS Inc. -> Abracon LLC; MPN ECS-320-8-37-CKM-TR3 -> ABS06-127-32.768KHZ-T; SKU 50-ECS-320-8-37-CKM-TR3CT-ND -> 535-14513-1-ND
Changed lines of the file:
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@@
       (effects (font (size 1.27 1.27)) hide)
     )
-    (property "Description" "32 MHz ±10ppm Crystal 8pF 60 Ohms 4-SMD, No Lead" (at 193.548 196.2404 0)
+    (property "Description" "32.768 kHz ±20ppm Crystal 12.5pF 90 kOhms 2-SMD, No Lead" (at 193.548 196.2404 0)
       (effects (font (size 1.27 1.27)) hide)
     )
-    (property "MFN" "ECS Inc." (at 193.548 196.2404 0)
+    (property "MFN" "Abracon LLC" (at 193.548 196.2404 0)
       (effects (font (size 1.27 1.27)) hide)
     )
-    (property "MPN" "ECS-320-8-37-CKM-TR3" (at 193.548 196.2404 0)
+    (property "MPN" "ABS06-127-32.768KHZ-T" (at 193.548 196.2404 0)
       (effects (font (size 1.27 1.27)) hide)
     )
-    (property "SKU" "50-ECS-320-8-37-CKM-TR3CT-ND" (at 193.548 196.2404 0)
+    (property "SKU" "535-14513-1-ND" (at 193.548 196.2404 0)
       (effects (font (size 1.27 1.27)) hide)
     )
