File: spirit_logger_hardware-backups/spirit_logger_hardware-2023-01-25_172253/CAN.kicad_sch (KiCad schematic)
At the start: 9 parts, among them U3 MCP25625-E/ML, Y1 16MHz

Commit message: drc and packaging
Parts:
- C23, C24: footprint MCU_Nordic_Accessory:C_0201 -> Capacitor_SMD.pretty:C_0402_1005Metric_Pad0.74x0.62mm_HandSolder
- C25, C26: footprint MCU_Nordic_Accessory:C_0201 -> Capacitor_SMD.pretty:C_0603_1608Metric
- R6: footprint Resistor_SMD:R_0201_0603Metric -> Resistor_SMD.pretty:R_0603_1608Metric
- TP5, TP6: footprint tuna-f1sh/jbr-kicad/Misc.pretty:TestPoint_Pad_D1.0mm_Tight -> tunaf1sh/misc.pretty:TestPoint_Pad_D1.0mm_Tight
- U3: footprint tuna-f1sh/jbr-kicad/QFN.pretty:QFN-28L -> tunaf1sh/QFN.pretty:QFN-28L
- Y1: footprint Crystal:Crystal_SMD_3225-4Pin_3.2x2.5mm -> Crystal.pretty:Crystal_SMD_3225-4Pin_3.2x2.5mm
Changed lines of the file:
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@@
       (effects (font (size 1.27 1.27)) (justify left) hide)
     )
-    (property "Footprint" "tuna-f1sh/jbr-kicad/Misc.pretty:TestPoint_Pad_D1.0mm_Tight" (id 2) (at 134.366 126.238 0)
+    (property "Footprint" "tunaf1sh/misc.pretty:TestPoint_Pad_D1.0mm_Tight" (id 2) (at 134.366 126.238 0)
       (effects (font (size 1.27 1.27)) hide)
     )
@@
       (effects (font (size 1.27 1.27)) (justify right))
     )
-    (property "Footprint" "Crystal:Crystal_SMD_3225-4Pin_3.2x2.5mm" (id 2) (at 212.598 69.088 0)
+    (property "Footprint" "Crystal.pretty:Crystal_SMD_3225-4Pin_3.2x2.5mm" (id 2) (at 212.598 69.088 0)
       (effects (font (size 1.27 1.27)) hide)
     )
@@
       (effects (font (size 1.27 1.27)) (justify left) hide)
     )
-    (property "Footprint" "tuna-f1sh/jbr-kicad/Misc.pretty:TestPoint_Pad_D1.0mm_Tight" (id 2) (at 180.848 95.504 0)
+    (property "Footprint" "tunaf1sh/misc.pretty:TestPoint_Pad_D1.0mm_Tight" (id 2) (at 180.848 95.504 0)
       (effects (font (size 1.27 1.27)) hide)
     )
@@
       (effects (font (size 1.27 1.27)) (justify left))
     )
-    (property "Footprint" "tuna-f1sh/jbr-kicad/QFN.pretty:QFN-28L" (id 2) (at 127.762 76.454 0)
+    (property "Footprint" "tunaf1sh/QFN.pretty:QFN-28L" (id 2) (at 127.762 76.454 0)
       (effects (font (size 1.27 1.27)) (justify bottom) hide)
     )
@@
       (effects (font (size 1.27 1.27)) (justify left))
     )
-    (property "Footprint" "MCU_Nordic_Accessory:C_0201" (id 2) (at 221.7928 65.278 0)
+    (property "Footprint" "Capacitor_SMD.pretty:C_0603_1608Metric" (id 2) (at 221.7928 65.278 0)
       (effects (font (size 1.27 1.27)) hide)
     )
@@
       (effects (font (size 1.27 1.27)) (justify left))
     )
-    (property "Footprint" "MCU_Nordic_Accessory:C_0201" (id 2) (at 189.0268 86.614 0)
+    (property "Footprint" "Capacitor_SMD.pretty:C_0402_1005Metric_Pad0.74x0.62mm_HandSolder" (id 2) (at 189.0268 86.614 0)
       (effects (font (size 1.27 1.27)) hide)
     )
@@
       (effects (font (size 1.27 1.27)) (justify left))
     )
-    (property "Footprint" "MCU_Nordic_Accessory:C_0201" (id 2) (at 211.6328 75.438 0)
+    (property "Footprint" "Capacitor_SMD.pretty:C_0603_1608Metric" (id 2) (at 211.6328 75.438 0)
       (effects (font (size 1.27 1.27)) hide)
     )
@@
       (effects (font (size 1.27 1.27)) (justify left))
     )
-    (property "Footprint" "Resistor_SMD:R_0201_0603Metric" (id 2) (at 107.188 73.406 0)
+    (property "Footprint" "Resistor_SMD.pretty:R_0603_1608Metric" (id 2) (at 107.188 73.406 0)
       (effects (font (size 1.27 1.27)) hide)
     )
@@
       (effects (font (size 1.27 1.27)) (justify left))
     )
-    (property "Footprint" "MCU_Nordic_Accessory:C_0201" (id 2) (at 106.2228 86.106 0)
-      (effects (font (size 1.27 1.27)) hide)
-    )
+    (property "Footprint" "Capacitor_SMD.pretty:C_0402_1005Metric_Pad0.74x0.62mm_HandSolder" (id 2) (at 106.2228 86.106 0)
+      (effects (font (size 1.27 1.27)) hide)
+    )
