File: spirit_logger_hardware-backups/spirit_logger_hardware-2023-01-25_172253/Radio.kicad_sch (KiCad schematic)
At the start: 29 parts, among them U1 nRF5340-QKAA, X1 Crystal_GND24, X2 Crystal

Commit message: drc and packaging
Parts:
- U1: footprint footprints_nordic:Nordic-AQFN-1EP_7x7mm_P0.4mm -> MCU_Nordic_Custom:Nordic-AQFN-1EP_7x7mm_P0.4mm; symbol MCU_Nordic_Custom:nRF5340-QKAA -> MCU_Nordic_Robb:nRF5340-QKAA
- U1: symbol MCU_Nordic_Custom:nRF5340-QKAA -> MCU_Nordic_Robb:nRF5340-QKAA
Connections:
- net VDD: now also C10.1, C11.1, C12.1, C13.1, C14.1, C15.1, C8.1, C9.1, U1.AC1 (VDD), U1.AG1 (VDD), U1.AJ31 (VDD), U1.AL11 (VDD), U1.AL17 (VDD), U1.AL25 (VDD), U1.AL3 (VDD), U1.AL7 (VDD), U1.B28 (VDD), U1.C1 (VDD), U1.E31 (VDD), U1.N31 (VDD), U1.U1 (VDD)
