File: spirit_logger_hardware-backups/spirit_logger_hardware-2023-01-25_172253/sensors.kicad_sch (KiCad schematic)
At the start: 15 parts, among them Q1 BSS123, U8 LSM6DSL

Commit message: drc and packaging
Parts:
- C36, C37: footprint MCU_Nordic_Accessory:C_0201 -> Capacitor_SMD.pretty:C_0402_1005Metric_Pad0.74x0.62mm_HandSolder
- D5: footprint Diode_SMD:D_SOD-323 -> Diode_SMD.pretty:D_SOD-323
- Q1: footprint Package_TO_SOT_SMD:SOT-23 -> Package_TO_SOT_SMD.pretty:SOT-23
- R14, R15, R16, R17, R18, R19, R20: footprint Resistor_SMD:R_0201_0603Metric -> Resistor_SMD.pretty:R_0402_1005Metric
- TP14, TP15, TP16: footprint TestPoint:TestPoint_Pad_D2.0mm -> TestPoint.pretty:TestPoint_Pad_D2.0mm
- U8: footprint Package_LGA:LGA-14_3x2.5mm_P0.5mm_LayoutBorder3x4y -> Package_LGA.pretty:LGA-14_3x2.5mm_P0.5mm_LayoutBorder3x4y
Connections:
- net VCC renamed VDD
Changed lines of the file:
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@@
     )
     (property "Footprint" "" (id 2) (at 226.3648 100.6348 0)
-      (effects (font (size 1.27 1.27)) hide)
+      (effects (font (size 1.524 1.524)))
     )
     (property "Datasheet" "" (id 3) (at 226.3648 100.6348 0)
-      (effects (font (size 1.27 1.27)) hide)
+      (effects (font (size 1.524 1.524)))
     )
     (pin "1")
@@
       (effects (font (size 1.27 1.27)) (justify left))
     )
-    (property "Footprint" "Resistor_SMD:R_0201_0603Metric" (id 2) (at 244.3988 96.5708 0)
+    (property "Footprint" "Resistor_SMD.pretty:R_0402_1005Metric" (id 2) (at 244.3988 96.5708 0)
       (effects (font (size 1.27 1.27)) hide)
     )
@@
       (effects (font (size 1.27 1.27)) (justify left))
     )
-    (property "Footprint" "MCU_Nordic_Accessory:C_0201" (id 2) (at 54.0004 77.216 0)
+    (property "Footprint" "Capacitor_SMD.pretty:C_0402_1005Metric_Pad0.74x0.62mm_HandSolder" (id 2) (at 54.0004 77.216 0)
       (effects (font (size 1.27 1.27)) hide)
     )
@@
     (pin "2")
   )
-  (symbol (lib_id "power:VCC") (at 91.3892 72.9488 0) (unit 1)
-    (in_bom yes) (on_board yes) (fields_autoplaced)
-    (property "Reference" "#PWR0151" (id 0) (at 91.3892 76.7588 0)
-      (effects (font (size 1.27 1.27)) hide)
-    )
-    (property "Value" "VCC" (id 1) (at 91.3892 69.373 0))
-    (property "Footprint" "" (id 2) (at 91.3892 72.9488 0)
-      (effects (font (size 1.27 1.27)) hide)
-    )
-    (property "Datasheet" "" (id 3) (at 91.3892 72.9488 0)
-      (effects (font (size 1.27 1.27)) hide)
-    )
-    (pin "1")
-  )
   (symbol (lib_id "Device:D_Zener") (at 188.976 99.1616 270) (unit 1)
     (in_bom yes) (on_board yes)
@@
       (effects (font (size 1.27 1.27)) (justify left))
     )
-    (property "Footprint" "Diode_SMD:D_SOD-323" (id 2) (at 188.976 99.1616 0)
+    (property "Footprint" "Diode_SMD.pretty:D_SOD-323" (id 2) (at 188.976 99.1616 0)
       (effects (font (size 1.27 1.27)) hide)
     )
@@
       (effects (font (size 1.27 1.27)) (justify left))
     )
-    (property "Footprint" "Resistor_SMD:R_0201_0603Metric" (id 2) (at 179.324 100.1776 0)
+    (property "Footprint" "Resistor_SMD.pretty:R_0402_1005Metric" (id 2) (at 179.324 100.1776 0)
       (effects (font (size 1.27 1.27)) hide)
     )
@@
       (effects (font (size 1.27 1.27)) (justify left) hide)
     )
-    (property "Footprint" "TestPoint:TestPoint_Pad_D2.0mm" (id 2) (at 249.4788 83.9724 0)
+    (property "Footprint" "TestPoint.pretty:TestPoint_Pad_D2.0mm" (id 2) (at 249.4788 83.9724 0)
       (effects (font (size 1.27 1.27)) hide)
     )
@@
     )
     (property "Footprint" "" (id 2) (at 244.3988 100.6348 0)
-      (effects (font (size 1.27 1.27)) hide)
+      (effects (font (size 1.524 1.524)))
     )
     (property "Datasheet" "" (id 3) (at 244.3988 100.6348 0)
-      (effects (font (size 1.27 1.27)) hide)
-    )
-    (pin "1")
-  )
-  (symbol (lib_id "power:GND") (at 54.9656 88.0364 0) (unit 1)
+      (effects (font (size 1.524 1.524)))
+    )
+    (pin "1")
+  )
+  (symbol (lib_id "power:VDD") (at 91.3892 72.9488 0) (unit 1)
+    (in_bom yes) (on_board yes) (fields_autoplaced)
+    (property "Reference" "#PWR0143" (id 0) (at 91.3892 76.7588 0)
+      (effects (font (size 1.27 1.27)) hide)
+    )
+    (property "Value" "VDD" (id 1) (at 91.3892 69.373 0))
+    (property "Footprint" "" (id 2) (at 91.3892 72.9488 0)
+      (effects (font (size 1.27 1.27)) hide)
+    )
+    (property "Datasheet" "" (id 3) (at 91.3892 72.9488 0)
+      (effects (font (size 1.27 1.27)) hide)
+    )
+    (pin "1")
+  )
+  (symbol (lib_name "GND_1") (lib_id "power:GND") (at 54.9656 88.0364 0) (unit 1)
     (in_bom yes) (on_board yes) (fields_autoplaced)
     (property "Reference" "#PWR0144" (id 0) (at 54.9656 94.3864 0)
@@
       (effects (font (size 1.27 1.27)) (justify left))
     )
-    (property "Footprint" "Resistor_SMD:R_0201_0603Metric" (id 2) (at 169.926 85.4456 0)
+    (property "Footprint" "Resistor_SMD.pretty:R_0402_1005Metric" (id 2) (at 169.926 85.4456 0)
       (effects (font (size 1.27 1.27)) hide)
     )
@@
     )
     (property "Footprint" "" (id 2) (at 169.926 105.5116 0)
-      (effects (font (size 1.27 1.27)) hide)
+      (effects (font (size 1.524 1.524)))
     )
     (property "Datasheet" "" (id 3) (at 169.926 105.5116 0)
-      (effects (font (size 1.27 1.27)) hide)
+      (effects (font (size 1.524 1.524)))
     )
     (pin "1")
@@
       (effects (font (size 1.27 1.27)) (justify left))
     )
-    (property "Footprint" "Resistor_SMD:R_0201_0603Metric" (id 2) (at 226.3648 88.6968 0)
+    (property "Footprint" "Resistor_SMD.pretty:R_0402_1005Metric" (id 2) (at 226.3648 88.6968 0)
       (effects (font (size 1.27 1.27)) hide)
     )
@@
       (effects (font (size 1.27 1.27)) (justify left))
     )
-    (property "Footprint" "Resistor_SMD:R_0201_0603Metric" (id 2) (at 195.326 95.3516 0)
+    (property "Footprint" "Resistor_SMD.pretty:R_0402_1005Metric" (id 2) (at 195.326 95.3516 0)
       (effects (font (size 1.27 1.27)) hide)
     )
@@
       (effects (font (size 1.27 1.27)) (justify left) hide)
     )
-    (property "Footprint" "TestPoint:TestPoint_Pad_D2.0mm" (id 2) (at 231.4448 83.8708 0)
+    (property "Footprint" "TestPoint.pretty:TestPoint_Pad_D2.0mm" (id 2) (at 231.4448 83.8708 0)
       (effects (font (size 1.27 1.27)) hide)
     )
@@
     (pin "1")
   )
-  (symbol (lib_id "power:GND") (at 91.3892 113.3348 0) (unit 1)
+  (symbol (lib_name "GND_1") (lib_id "power:GND") (at 91.3892 113.3348 0) (unit 1)
     (in_bom yes) (on_board yes) (fields_autoplaced)
     (property "Reference" "#PWR0145" (id 0) (at 91.3892 119.6848 0)
@@
       (effects (font (size 1.27 1.27)) (justify left))
     )
-    (property "Footprint" "MCU_Nordic_Accessory:C_0201" (id 2) (at 41.148 77.216 0)
+    (property "Footprint" "Capacitor_SMD.pretty:C_0402_1005Metric_Pad0.74x0.62mm_HandSolder" (id 2) (at 41.148 77.216 0)
       (effects (font (size 1.27 1.27)) hide)
     )
@@
       (effects (font (size 1.27 1.27)) (justify left))
     )
-    (property "Footprint" "Resistor_SMD:R_0201_0603Metric" (id 2) (at 244.3988 88.6968 0)
+    (property "Footprint" "Resistor_SMD.pretty:R_0402_1005Metric" (id 2) (at 244.3988 88.6968 0)
       (effects (font (size 1.27 1.27)) hide)
     )
@@
       (effects (font (size 1.27 1.27)) (justify left))
     )
-    (property "Footprint" "Resistor_SMD:R_0201_0603Metric" (id 2) (at 226.3648 96.5708 0)
+    (property "Footprint" "Resistor_SMD.pretty:R_0402_1005Metric" (id 2) (at 226.3648 96.5708 0)
       (effects (font (size 1.27 1.27)) hide)
     )
@@
       (effects (font (size 1.27 1.27)) (justify left))
     )
-    (property "Footprint" "Package_TO_SOT_SMD:SOT-23" (id 2) (at 167.386 97.2566 0)
+    (property "Footprint" "Package_TO_SOT_SMD.pretty:SOT-23" (id 2) (at 167.386 97.2566 0)
       (effects (font (size 1.27 1.27) italic) (justify left) hide)
     )
@@
       (effects (font (size 1.27 1.27)) (justify left) hide)
     )
-    (property "Footprint" "TestPoint:TestPoint_Pad_D2.0mm" (id 2) (at 198.882 100.4316 0)
+    (property "Footprint" "TestPoint.pretty:TestPoint_Pad_D2.0mm" (id 2) (at 198.882 100.4316 0)
       (effects (font (size 1.27 1.27)) hide)
     )
@@
     (property "Reference" "U8" (id 0) (at 106.5937 79.8915 0))
     (property "Value" "LSM6DSL" (id 1) (at 106.5937 82.4284 0))
-    (property "Footprint" "Package_LGA:LGA-14_3x2.5mm_P0.5mm_LayoutBorder3x4y" (id 2) (at 78.6892 110.998 0)
+    (property "Footprint" "Package_LGA.pretty:LGA-14_3x2.5mm_P0.5mm_LayoutBorder3x4y" (id 2) (at 78.6892 110.998 0)
       (effects (font (size 1.27 1.27)) (justify left) hide)
     )
