File: spirit_logger_hardware-backups/spirit_logger_hardware-2023-01-25_172253/spirit_logger_hardware.kicad_sch (KiCad schematic)
At the start: 27 parts, among them J1 PicoBlade, J2 PicoBlade, U2 MX25R6435F

Commit message: drc and packaging
Parts:
- removed TP26: TestPoint, tuna-f1sh/jbr-kicad/Misc.pretty:TestPoint_Pad_D1.0mm_Tight, symbol Connector:TestPoint_Small
- D2: footprint LED_SMD:LED_Kingbright_AAA3528ESGCT -> LED_SMD.pretty:LED_Kingbright_AAA3528ESGCT
- D3: footprint Package_TO_SOT_SMD:SOT-23 -> Package_TO_SOT_SMD.pretty:SOT-23
- J1, J2: footprint Connector_Molex:Molex_PicoBlade_53261-0571_1x05-1MP_P1.25mm_Horizontal -> Connector_Molex.pretty:Molex_PicoBlade_53261-0571_1x05-1MP_P1.25mm_Horizontal
- JP1: footprint Jumper:SolderJumper-2_P1.3mm_Open_RoundedPad1.0x1.5mm -> Jumper.pretty:SolderJumper-2_P1.3mm_Open_RoundedPad1.0x1.5mm
- R2, R3, R4: footprint Resistor_SMD:R_0201_0603Metric -> Resistor_SMD.pretty:R_0402_1005Metric
- R5: footprint Resistor_SMD:R_0603_1608Metric -> Resistor_SMD.pretty:R_0603_1608Metric
- TP1, TP2, TP3, TP4: footprint tuna-f1sh/jbr-kicad/Misc.pretty:TestPoint_Pad_D1.0mm_Tight -> tunaf1sh/misc.pretty:TestPoint_Pad_D1.0mm_Tight
- TP?: renamed from TP19; footprint tuna-f1sh/jbr-kicad/Misc.pretty:TestPoint_Pad_D1.0mm_Tight -> tunaf1sh/misc.pretty:TestPoint_Pad_D1.0mm_Tight
- TP?: renamed from TP23; footprint tuna-f1sh/jbr-kicad/Misc.pretty:TestPoint_Pad_D1.0mm_Tight -> tunaf1sh/misc.pretty:TestPoint_Pad_D1.0mm_Tight
- TP?: renamed from TP18; footprint tuna-f1sh/jbr-kicad/Misc.pretty:TestPoint_Pad_D1.0mm_Tight -> tunaf1sh/misc.pretty:TestPoint_Pad_D1.0mm_Tight
- TP?: renamed from TP21; footprint tuna-f1sh/jbr-kicad/Misc.pretty:TestPoint_Pad_D1.0mm_Tight -> tunaf1sh/misc.pretty:TestPoint_Pad_D1.0mm_Tight
- TP?: renamed from TP20; footprint tuna-f1sh/jbr-kicad/Misc.pretty:TestPoint_Pad_D1.0mm_Tight -> tunaf1sh/misc.pretty:TestPoint_Pad_D1.0mm_Tight
- TP?: renamed from TP25; footprint tuna-f1sh/jbr-kicad/Misc.pretty:TestPoint_Pad_D1.0mm_Tight -> tunaf1sh/misc.pretty:TestPoint_Pad_D1.0mm_Tight
- TP?: renamed from TP17; footprint tuna-f1sh/jbr-kicad/Misc.pretty:TestPoint_Pad_D1.0mm_Tight -> tunaf1sh/misc.pretty:TestPoint_Pad_D1.0mm_Tight
- TP?: renamed from TP24; footprint tuna-f1sh/jbr-kicad/Misc.pretty:TestPoint_Pad_D1.0mm_Tight -> tunaf1sh/misc.pretty:TestPoint_Pad_D1.0mm_Tight
- TP?: renamed from TP22; footprint tuna-f1sh/jbr-kicad/Misc.pretty:TestPoint_Pad_D1.0mm_Tight -> tunaf1sh/misc.pretty:TestPoint_Pad_D1.0mm_Tight
- U2: footprint Package_SON:WSON-8-1EP_6x5mm_P1.27mm_EP3.4x4mm -> Package_SON.pretty:WSON-8-1EP_6x5mm_P1.27mm_EP3.4x4mm
Connections:
- net P0.19/SDA renamed P0.19/I2C
- net P0.21/SCL renamed P0.21/I2C
- net VCC renamed VDD
